File: hard/kicad/durango/cpu/cpu.sch (KiCad schematic (older format))
At the start: 15 parts, among them U1 65SC02, U10 4040, U11 74LS30, U2 62256, U3 27C128, U4 74HC139, U5 74HC139, U6 74HC139, U7 74HC374, U8 74HC74, U9 74HC245, X1 1 MHz

Commit message: work on durango proto CPU board
Parts:
- added C1: 100n, symbol Device:C
- added D1: 1N4148, symbol Device:D
- added J1: NANOLINK, symbol Connector_Generic:Conn_01x03
- added J2: IO9 INPUT, symbol Connector_Generic:Conn_01x09
- added Q1, Q2: BC547, Package_TO_SOT_THT:TO-92_Inline, symbol Transistor_BJT:BC547
- added R1, R2: 22K, symbol Device:R
- added R3: 1K, symbol Device:R
- added RN1: 4K7, Resistor_THT:R_Array_SIP5, symbol Device:R_Network04
- added SW1: RESET, symbol Switch:SW_Push
- U11: value 74LS30 -> 74HC30
- renumbered D1 to D2, R1 to R4, RN1 to RN2
Connections:
- net labels added: +5V, A0, A1, A10, A11, A12, A13, A14, A15, A2, A3, A4, A5, A6, A7, A8, A9, D0, D1, D2, D3, D4, D5, D6, D7, GND, SERCLK, SERDAT
- wire segments 0 -> 144
- no-connect marks 0 -> 8
Other:
- moved on the sheet: R4, U11A, U8A, U8B

Commit message: working on cpu schematic at iMac
Parts:
- C1: symbol Device:C -> cpu-rescue:C-Device
- D1: symbol Device:D -> cpu-rescue:D-Device
- D2: symbol Device:LED -> cpu-rescue:LED-Device
- J1: symbol Connector_Generic:Conn_01x03 -> cpu-rescue:Conn_01x03-Connector_Generic
- J2: symbol Connector_Generic:Conn_01x09 -> cpu-rescue:Conn_01x09-Connector_Generic
- Q1, Q2: symbol Transistor_BJT:BC547 -> cpu-rescue:BC547-Transistor_BJT
- R1, R2, R3: symbol Device:R -> cpu-rescue:R-Device
- R4: value R -> 390; symbol Device:R -> cpu-rescue:R-Device
- RN1: symbol Device:R_Network04 -> cpu-rescue:R_Network04-Device
- RN2: symbol Device:R_Pack04_SIP -> cpu-rescue:R_Pack04_SIP-Device
- SW1: symbol Switch:SW_Push -> cpu-rescue:SW_Push-Switch
- U1: symbol CPU:MOS6502 -> cpu-rescue:MOS6502-CPU
- U10: symbol 4xxx:4040 -> cpu-rescue:4040-4xxx
- U11: symbol 74xx:74LS30 -> cpu-rescue:74LS30-74xx
- U2: symbol Memory_RAM:62256 -> cpu-rescue:62256-Memory_RAM
- U3: symbol Memory_EPROM:27C128 -> cpu-rescue:27C128-Memory_EPROM
- U4, U5, U6: symbol 74xx:74LS139 -> cpu-rescue:74LS139-74xx
- U7: symbol 74xx:74HC374 -> cpu-rescue:74HC374-74xx
- U8: symbol 74xx:74HC74 -> cpu-rescue:74HC74-74xx
- U9: symbol 74xx:74HC245 -> cpu-rescue:74HC245-74xx
- X1: symbol Oscillator:ACO-xxxMHz -> cpu-rescue:ACO-xxxMHz-Oscillator
Connections:
- net labels added: +5V-power, BUZ, DI0, DI1, DI2, DI3, GND-power, IEN, ~IO8Q, ~IO8U, ~IO9Q, ~IOAQ, ~IOBQ, ~LTC, ~RES
- wire segments 144 -> 211
- no-connect marks 8 -> 20

Commit message: messing with KiCAD
Parts:
- C1: symbol cpu-rescue:C-Device -> cpu-rescue:C-Device-cpu-rescue
- D1: symbol cpu-rescue:D-Device -> cpu-rescue:D-Device-cpu-rescue
- D2: symbol cpu-rescue:LED-Device -> cpu-rescue:LED-Device-cpu-rescue
- J1: symbol cpu-rescue:Conn_01x03-Connector_Generic -> cpu-rescue:Conn_01x03-Connector_Generic-cpu-rescue
- J2: symbol cpu-rescue:Conn_01x09-Connector_Generic -> cpu-rescue:Conn_01x09-Connector_Generic-cpu-rescue
- Q1, Q2: symbol cpu-rescue:BC547-Transistor_BJT -> cpu-rescue:BC547-Transistor_BJT-cpu-rescue
- R1, R2, R3, R4: symbol cpu-rescue:R-Device -> cpu-rescue:R-Device-cpu-rescue
- RN1: symbol cpu-rescue:R_Network04-Device -> cpu-rescue:R_Network04-Device-cpu-rescue
- RN2: symbol cpu-rescue:R_Pack04_SIP-Device -> cpu-rescue:R_Pack04_SIP-Device-cpu-rescue
- SW1: symbol cpu-rescue:SW_Push-Switch -> cpu-rescue:SW_Push-Switch-cpu-rescue
- U1: symbol cpu-rescue:MOS6502-CPU -> cpu-rescue:MOS6502-CPU-cpu-rescue
- U10: symbol cpu-rescue:4040-4xxx -> cpu-rescue:4040-4xxx-cpu-rescue
- U11: symbol cpu-rescue:74LS30-74xx -> cpu-rescue:74LS30-74xx-cpu-rescue
- U2: symbol cpu-rescue:62256-Memory_RAM -> cpu-rescue:62256-Memory_RAM-cpu-rescue
- U3: symbol cpu-rescue:27C128-Memory_EPROM -> cpu-rescue:27C128-Memory_EPROM-cpu-rescue
- U4, U5, U6: symbol cpu-rescue:74LS139-74xx -> cpu-rescue:74LS139-74xx-cpu-rescue
- U7: symbol cpu-rescue:74HC374-74xx -> cpu-rescue:74HC374-74xx-cpu-rescue
- U8: symbol cpu-rescue:74HC74-74xx -> cpu-rescue:74HC74-74xx-cpu-rescue
- U9: symbol cpu-rescue:74HC245-74xx -> cpu-rescue:74HC245-74xx-cpu-rescue
- X1: symbol cpu-rescue:ACO-xxxMHz-Oscillator -> cpu-rescue:ACO-xxxMHz-Oscillator-cpu-rescue
Connections:
- net labels removed: +5V-power
- wire segments 211 -> 212

Commit message: mostly finished Durango CPU board
Parts:
- removed J2: IO9 INPUT, symbol cpu-rescue:Conn_01x09-Connector_Generic-cpu-rescue
- added BZ1: Buzzer, symbol Device:Buzzer
- added D3, D4: 1N4148, Diode_THT:D_DO-35_SOD27_P7.62mm_Horizontal, symbol Diode:1N4148
- added J2: IO9 INPUT, symbol Connector_Generic:Conn_01x10
- added J3: IO8 PORT, symbol Connector_Generic:Conn_01x13
- added Q3: BC547, Package_TO_SOT_THT:TO-92_Inline, symbol Transistor_BJT:BC547
- added R5: 22, symbol Device:R
- added RN3: 220K, Resistor_THT:R_Array_SIP9, symbol Device:R_Network08
- C1: symbol cpu-rescue:C-Device-cpu-rescue -> cpu-rescue:C-Device-cpu-rescue-cpu-rescue
- D1: symbol cpu-rescue:D-Device-cpu-rescue -> cpu-rescue:D-Device-cpu-rescue-cpu-rescue
- D2: value RED LED -> INT. DISABLED; symbol cpu-rescue:LED-Device-cpu-rescue -> cpu-rescue:LED-Device-cpu-rescue-cpu-rescue
- J1: symbol cpu-rescue:Conn_01x03-Connector_Generic-cpu-rescue -> cpu-rescue:Conn_01x03-Connector_Generic-cpu-rescue-cpu-rescue
- Q1, Q2: symbol cpu-rescue:BC547-Transistor_BJT-cpu-rescue -> cpu-rescue:BC547-Transistor_BJT-cpu-rescue-cpu-rescue
- R1, R2, R3, R4: symbol cpu-rescue:R-Device-cpu-rescue -> cpu-rescue:R-Device-cpu-rescue-cpu-rescue
- RN1: symbol cpu-rescue:R_Network04-Device-cpu-rescue -> cpu-rescue:R_Network04-Device-cpu-rescue-cpu-rescue
- RN2: symbol cpu-rescue:R_Pack04_SIP-Device-cpu-rescue -> cpu-rescue:R_Pack04_SIP-Device-cpu-rescue-cpu-rescue
- SW1: symbol cpu-rescue:SW_Push-Switch-cpu-rescue -> cpu-rescue:SW_Push-Switch-cpu-rescue-cpu-rescue
- U1: symbol cpu-rescue:MOS6502-CPU-cpu-rescue -> cpu-rescue:MOS6502-CPU-cpu-rescue-cpu-rescue
- U10: symbol cpu-rescue:4040-4xxx-cpu-rescue -> cpu-rescue:4040-4xxx-cpu-rescue-cpu-rescue
- U11: symbol cpu-rescue:74LS30-74xx-cpu-rescue -> cpu-rescue:74LS30-74xx-cpu-rescue-cpu-rescue
- U2: symbol cpu-rescue:62256-Memory_RAM-cpu-rescue -> cpu-rescue:62256-Memory_RAM-cpu-rescue-cpu-rescue
- U3: symbol cpu-rescue:27C128-Memory_EPROM-cpu-rescue -> cpu-rescue:27C128-Memory_EPROM-cpu-rescue-cpu-rescue
- U4, U5, U6: symbol cpu-rescue:74LS139-74xx-cpu-rescue -> cpu-rescue:74LS139-74xx-cpu-rescue-cpu-rescue
- U7: symbol cpu-rescue:74HC374-74xx-cpu-rescue -> cpu-rescue:74HC374-74xx-cpu-rescue-cpu-rescue
- U8: symbol cpu-rescue:74HC74-74xx-cpu-rescue -> cpu-rescue:74HC74-74xx-cpu-rescue-cpu-rescue
- U9: symbol cpu-rescue:74HC245-74xx-cpu-rescue -> cpu-rescue:74HC245-74xx-cpu-rescue-cpu-rescue
- X1: symbol cpu-rescue:ACO-xxxMHz-Oscillator-cpu-rescue -> cpu-rescue:ACO-xxxMHz-Oscillator-cpu-rescue-cpu-rescue
Connections:
- net +5V: now also U1.38 (~SO), U2.28 (VCC), J2.1 (Pin_1), Q3.1 (C)
- net A0: now also J3.1 (Pin_1)
- net A1: now also J3.2 (Pin_2)
- net D0: now also U7.3 (D0), U9.14 (B4), J3.3 (Pin_3)
- net D1: now also U7.4 (D1), U9.13 (B5), J3.4 (Pin_4)
- net D2: now also U7.7 (D2), U9.12 (B6), J3.5 (Pin_5)
- net D3: now also U7.8 (D3), U9.11 (B7), J3.6 (Pin_6)
- net D4: now also U7.13 (D4), U9.15 (B3), J3.7 (Pin_7)
- net D5: now also U7.14 (D5), U9.16 (B2), J3.8 (Pin_8)
- net D6: now also U7.17 (D6), U9.17 (B1), J3.9 (Pin_9)
- net D7: now also U7.18 (D7), U9.18 (B0), J3.10 (Pin_10)
- net DI0: now also J2.6 (Pin_6), RN3.5 (R4)
- net DI1: now also J2.7 (Pin_7), RN3.4 (R3)
- net DI2: now also J2.8 (Pin_8), RN3.3 (R2)
- net DI3: now also J2.9 (Pin_9), RN3.2 (R1)
- net GND: now also U1.1 (VSS), U1.21 (VSS), U2.14 (GND), U3.14 (GND), J2.10 (Pin_10), J3.13 (Pin_13), R5.1, RN3.1 (common)
- net ~IO8Q: now also U6.12 (O0), J3.12 (Pin_12)
- net ~IO8U: now also U5.4 (O0), J3.11 (Pin_11)
- net at U1.39 (Phi2.OUT), U10.10 (CLK), U4.14 (A0): now also X1.7 (GND)
- net DI7: now reaches U9.2 (A0)
- net DI7: now also J2.2 (Pin_2), RN3.9 (R8)
- net DI6: now reaches U9.3 (A1)
- net DI6: now also J2.3 (Pin_3), RN3.8 (R7)
- net DI5: now reaches U9.4 (A2)
- net DI5: now also J2.4 (Pin_4), RN3.7 (R6)
- net DI4: now reaches U9.5 (A3)
- net DI4: now also J2.5 (Pin_5), RN3.6 (R5)
- net at U8.5 (Q): now also D3.2 (A)
- net ~IO9Q: no longer names the net of U6.11 (O1), U9.19 (CE)
- net ~IOAQ: no longer names the net of U6.10 (O2), U8.11 (C)
- net ~IOBQ: no longer names the net of U6.9 (O3), U8.3 (C)
- net ~LTC: no longer names the net of U6.6 (O2), U7.11 (Cp)
- net ~RES: no longer names the net of C1.1, R3.2, SW1.2, U1.40 (~RESET), U8.1 (~R), U8.13 (~R)
- new net: D3.1 (K), D4.1 (K), Q3.2 (B)
- new net: BZ1.1 (-), Q3.3 (E)
- new net: BZ1.2 (+), R5.2
- no-connect marks 20 -> 21
Other:
- moved on the sheet: D2, R4, U7, U8A, U8B, U9, X1

Commit message: Durango CPU board ready
Parts:
- added U12: LTC4622G, symbol Display_Character:LTC4622G
- C1: symbol cpu-rescue:C-Device-cpu-rescue-cpu-rescue -> cpu-rescue:C-Device-cpu-rescue-cpu-rescue-cpu-rescue
- D1: symbol cpu-rescue:D-Device-cpu-rescue-cpu-rescue -> cpu-rescue:D-Device-cpu-rescue-cpu-rescue-cpu-rescue
- D2: symbol cpu-rescue:LED-Device-cpu-rescue-cpu-rescue -> cpu-rescue:LED-Device-cpu-rescue-cpu-rescue-cpu-rescue
- J1: symbol cpu-rescue:Conn_01x03-Connector_Generic-cpu-rescue-cpu-rescue -> cpu-rescue:Conn_01x03-Connector_Generic-cpu-rescue-cpu-rescue-cpu-rescue
- Q1, Q2: symbol cpu-rescue:BC547-Transistor_BJT-cpu-rescue-cpu-rescue -> cpu-rescue:BC547-Transistor_BJT-cpu-rescue-cpu-rescue-cpu-rescue
- R1, R2, R3, R4: symbol cpu-rescue:R-Device-cpu-rescue-cpu-rescue -> cpu-rescue:R-Device-cpu-rescue-cpu-rescue-cpu-rescue
- RN1: symbol cpu-rescue:R_Network04-Device-cpu-rescue-cpu-rescue -> cpu-rescue:R_Network04-Device-cpu-rescue-cpu-rescue-cpu-rescue
- RN2: symbol cpu-rescue:R_Pack04_SIP-Device-cpu-rescue-cpu-rescue -> cpu-rescue:R_Pack04_SIP-Device-cpu-rescue-cpu-rescue-cpu-rescue
- SW1: symbol cpu-rescue:SW_Push-Switch-cpu-rescue-cpu-rescue -> cpu-rescue:SW_Push-Switch-cpu-rescue-cpu-rescue-cpu-rescue
- U1: symbol cpu-rescue:MOS6502-CPU-cpu-rescue-cpu-rescue -> cpu-rescue:MOS6502-CPU-cpu-rescue-cpu-rescue-cpu-rescue
- U10: symbol cpu-rescue:4040-4xxx-cpu-rescue-cpu-rescue -> cpu-rescue:4040-4xxx-cpu-rescue-cpu-rescue-cpu-rescue
- U11: symbol cpu-rescue:74LS30-74xx-cpu-rescue-cpu-rescue -> cpu-rescue:74LS30-74xx-cpu-rescue-cpu-rescue-cpu-rescue
- U2: symbol cpu-rescue:62256-Memory_RAM-cpu-rescue-cpu-rescue -> cpu-rescue:62256-Memory_RAM-cpu-rescue-cpu-rescue-cpu-rescue
- U3: symbol cpu-rescue:27C128-Memory_EPROM-cpu-rescue-cpu-rescue -> cpu-rescue:27C128-Memory_EPROM-cpu-rescue-cpu-rescue-cpu-rescue
- U4, U5, U6: symbol cpu-rescue:74LS139-74xx-cpu-rescue-cpu-rescue -> cpu-rescue:74LS139-74xx-cpu-rescue-cpu-rescue-cpu-rescue
- U7: symbol cpu-rescue:74HC374-74xx-cpu-rescue-cpu-rescue -> cpu-rescue:74HC374-74xx-cpu-rescue-cpu-rescue-cpu-rescue
- U8: symbol cpu-rescue:74HC74-74xx-cpu-rescue-cpu-rescue -> cpu-rescue:74HC74-74xx-cpu-rescue-cpu-rescue-cpu-rescue
- U9: symbol cpu-rescue:74HC245-74xx-cpu-rescue-cpu-rescue -> cpu-rescue:74HC245-74xx-cpu-rescue-cpu-rescue-cpu-rescue
- X1: symbol cpu-rescue:ACO-xxxMHz-Oscillator-cpu-rescue-cpu-rescue -> cpu-rescue:ACO-xxxMHz-Oscillator-cpu-rescue-cpu-rescue-cpu-rescue
Connections:
- net at U7.12 (O4): now also RN2.8 (R4.2)
- net at U7.15 (O5): now also RN2.6 (R3.2)
- net at U7.16 (O6): now also RN2.4 (R2.2)
- net at U7.19 (O7): now also RN2.2 (R1.2)
- net at U7.2 (O0): now also U12.9 (CA1L)
- net at U7.5 (O1): now also U12.8 (CA1R)
- net at U7.6 (O2): now also U12.7 (CA2L)
- net at U7.9 (O3): now also U12.6 (CA2R)
- net at RN2.1 (R1.1): now also U12.2 (A/D)
- net at RN2.3 (R2.1): now also U12.3 (B/E)
- net at RN2.5 (R3.1): now also U12.4 (C/F)
- net at RN2.7 (R4.1): now also U12.5 (D.P./G)
- no-connect marks 21 -> 22
Other:
- moved on the sheet: RN2

Commit message: routing durango CPU board
Parts:
- BZ1: footprint (none) -> Buzzer_Beeper:Buzzer_12x9.5RM7.6
- C1: footprint (none) -> Capacitor_THT:C_Rect_L10.0mm_W5.0mm_P5.00mm_P7.50mm
- D1: footprint (none) -> Diode_THT:D_DO-34_SOD68_P2.54mm_Vertical_AnodeUp
- D2: footprint (none) -> LED_THT:LED_D3.0mm
- J1: footprint (none) -> Connector_PinHeader_2.54mm:PinHeader_1x03_P2.54mm_Vertical
- J2: footprint (none) -> Connector_PinHeader_2.54mm:PinHeader_1x10_P2.54mm_Vertical
- J3: footprint (none) -> Connector_PinHeader_2.54mm:PinHeader_1x13_P2.54mm_Vertical
- R1, R2, R3, R4, R5: footprint (none) -> Resistor_THT:R_Axial_DIN0204_L3.6mm_D1.6mm_P2.54mm_Vertical
- SW1: footprint (none) -> Button_Switch_THT:KSA_Tactile_SPST
- U10, U4, U5, U6: footprint (none) -> Package_DIP:DIP-16_W7.62mm
- U11, U8: footprint (none) -> Package_DIP:DIP-14_W7.62mm
- U12: footprint (none) -> Connector_PinHeader_2.54mm:PinHeader_1x09_P2.54mm_Vertical
- U2: footprint (none) -> Package_DIP:DIP-28_W15.24mm
- U7, U9: footprint (none) -> Package_DIP:DIP-20_W7.62mm
Changed lines of the file:
@@
 F 0 "U2" H 3650 3150 50  0000 C CNN
 F 1 "62256" H 4050 3150 50  0000 C CNN
-F 2 "" H 3850 2050 50  0001 C CNN
+F 2 "Package_DIP:DIP-28_W15.24mm" H 3850 2050 50  0001 C CNN
 F 3 "http://www.6502.org/users/alexis/62256.pdf" H 3850 2050 50  0001 C CNN
 	1    3850 2050
@@
 F 0 "U4" H 3750 4517 50  0000 C CNN
 F 1 "74HC139" H 3750 4426 50  0000 C CNN
-F 2 "" H 3750 4150 50  0001 C CNN
+F 2 "Package_DIP:DIP-16_W7.62mm" H 3750 4150 50  0001 C CNN
 F 3 "http://www.ti.com/lit/gpn/sn74LS139" H 3750 4150 50  0001 C CNN
 	1    3750 4150
@@
 F 0 "U4" H 3750 5267 50  0000 C CNN
 F 1 "74HC139" H 3750 5176 50  0000 C CNN
-F 2 "" H 3750 4900 50  0001 C CNN
+F 2 "Package_DIP:DIP-16_W7.62mm" H 3750 4900 50  0001 C CNN
 F 3 "http://www.ti.com/lit/gpn/sn74LS139" H 3750 4900 50  0001 C CNN
 	2    3750 4900
@@
 F 0 "U5" H 5300 4750 50  0000 C CNN
 F 1 "74HC139" H 5300 4850 50  0000 C CNN
-F 2 "" H 5300 4500 50  0001 C CNN
+F 2 "Package_DIP:DIP-16_W7.62mm" H 5300 4500 50  0001 C CNN
 F 3 "http://www.ti.com/lit/gpn/sn74LS139" H 5300 4500 50  0001 C CNN
 	1    5300 4500
@@
 F 0 "U5" H 5300 3350 50  0000 C CNN
 F 1 "74HC139" H 5300 3250 50  0000 C CNN
-F 2 "" H 5300 3700 50  0001 C CNN
+F 2 "Package_DIP:DIP-16_W7.62mm" H 5300 3700 50  0001 C CNN
 F 3 "http://www.ti.com/lit/gpn/sn74LS139" H 5300 3700 50  0001 C CNN
 	2    5300 3700
@@
 F 0 "U10" H 1200 5550 50  0000 C CNN
 F 1 "4040" H 1200 5450 50  0000 C CNN
-F 2 "" H 1050 4750 50  0001 C CNN
+F 2 "Package_DIP:DIP-16_W7.62mm" H 1050 4750 50  0001 C CNN
 F 3 "http://www.intersil.com/content/dam/Intersil/documents/cd40/cd4020bms-24bms-40bms.pdf" H 1050 4750 50  0001 C CNN
 	1    1050 4750
@@
 F 0 "U6" H 5300 5717 50  0000 C CNN
 F 1 "74HC139" H 5300 5626 50  0000 C CNN
-F 2 "" H 5300 5350 50  0001 C CNN
+F 2 "Package_DIP:DIP-16_W7.62mm" H 5300 5350 50  0001 C CNN
 F 3 "http://www.ti.com/lit/gpn/sn74LS139" H 5300 5350 50  0001 C CNN
 	1    5300 5350
@@
 F 0 "U6" H 5350 6467 50  0000 C CNN
 F 1 "74HC139" H 5350 6376 50  0000 C CNN
-F 2 "" H 5350 6100 50  0001 C CNN
+F 2 "Package_DIP:DIP-16_W7.62mm" H 5350 6100 50  0001 C CNN
 F 3 "http://www.ti.com/lit/gpn/sn74LS139" H 5350 6100 50  0001 C CNN
 	2    5350 6100
@@
 F 0 "U9" H 6950 6431 50  0000 C CNN
 F 1 "74HC245" H 6950 6340 50  0000 C CNN
-F 2 "" H 6950 5450 50  0001 C CNN
+F 2 "Package_DIP:DIP-20_W7.62mm" H 6950 5450 50  0001 C CNN
 F 3 "http://www.ti.com/lit/gpn/sn74HC245" H 6950 5450 50  0001 C CNN
 	1    6950 5450
@@
 F 0 "U7" H 3900 6850 50  0000 C CNN
 F 1 "74HC374" H 3550 6850 50  0000 C CNN
-F 2 "" H 3750 6200 50  0001 C CNN
+F 2 "Package_DIP:DIP-20_W7.62mm" H 3750 6200 50  0001 C CNN
 F 3 "https://www.ti.com/lit/ds/symlink/cd74hct374.pdf" H 3750 6200 50  0001 C CNN
 	1    3750 6200
@@
 F 0 "U8" H 6750 2081 50  0000 C CNN
 F 1 "74HC74" H 6750 1990 50  0000 C CNN
-F 2 "" H 6750 1600 50  0001 C CNN
+F 2 "Package_DIP:DIP-14_W7.62mm" H 6750 1600 50  0001 C CNN
 F 3 "74xx/74hc_hct74.pdf" H 6750 1600 50  0001 C CNN
 	1    6750 1600
@@
 F 0 "U8" H 6750 3031 50  0000 C CNN
 F 1 "74HC74" H 6750 2940 50  0000 C CNN
-F 2 "" H 6750 2550 50  0001 C CNN
+F 2 "Package_DIP:DIP-14_W7.62mm" H 6750 2550 50  0001 C CNN
 F 3 "74xx/74hc_hct74.pdf" H 6750 2550 50  0001 C CNN
 	2    6750 2550
@@
 F 0 "D2" H 7600 2400 50  0000 C CNN
 F 1 "INT. DISABLED" H 7550 2500 50  0000 C CNN
-F 2 "" H 7600 2650 50  0001 C CNN
+F 2 "LED_THT:LED_D3.0mm" H 7600 2650 50  0001 C CNN
 F 3 "~" H 7600 2650 50  0001 C CNN
 	1    7600 2650
@@
 F 0 "R4" V 7400 2600 50  0000 L CNN
 F 1 "390" V 7200 2600 50  0000 L CNN
-F 2 "" V 7230 2650 50  0001 C CNN
+F 2 "Resistor_THT:R_Axial_DIN0204_L3.6mm_D1.6mm_P2.54mm_Vertical" V 7230 2650 50  0001 C CNN
 F 3 "~" H 7300 2650 50  0001 C CNN
 	1    7300 2650
@@
 F 0 "U11" H 2250 5150 50  0000 C CNN
 F 1 "74HC30" H 2200 5250 50  0000 C CNN
-F 2 "" H 2150 4950 50  0001 C CNN
+F 2 "Package_DIP:DIP-14_W7.62mm" H 2150 4950 50  0001 C CNN
 F 3 "http://www.ti.com/lit/gpn/sn74LS30" H 2150 4950 50  0001 C CNN
 	1    2150 4950
@@
 F 0 "R2" H 850 2300 50  0000 L CNN
 F 1 "22K" H 700 2100 50  0000 L CNN
-F 2 "" V 730 2250 50  0001 C CNN
+F 2 "Resistor_THT:R_Axial_DIN0204_L3.6mm_D1.6mm_P2.54mm_Vertical" V 730 2250 50  0001 C CNN
 F 3 "~" H 800 2250 50  0001 C CNN
 	1    800  2250
@@
 F 0 "R1" H 650 2300 50  0000 L CNN
 F 1 "22K" H 500 2100 50  0000 L CNN
-F 2 "" V 530 2250 50  0001 C CNN
+F 2 "Resistor_THT:R_Axial_DIN0204_L3.6mm_D1.6mm_P2.54mm_Vertical" V 530 2250 50  0001 C CNN
 F 3 "~" H 600 2250 50  0001 C CNN
 	1    600  2250
@@
 F 0 "J1" V 900 1700 50  0000 R CNN
 F 1 "NANOLINK" V 800 1850 50  0000 R CNN
-F 2 "" H 700 1650 50  0001 C CNN
+F 2 "Connector_PinHeader_2.54mm:PinHeader_1x03_P2.54mm_Vertical" H 700 1650 50  0001 C CNN
 F 3 "~" H 700 1650 50  0001 C CNN
 	1    700  1650
@@
 F 0 "R3" V 1043 850 50  0000 C CNN
 F 1 "1K" V 1134 850 50  0000 C CNN
-F 2 "" V 1180 850 50  0001 C CNN
+F 2 "Resistor_THT:R_Axial_DIN0204_L3.6mm_D1.6mm_P2.54mm_Vertical" V 1180 850 50  0001 C CNN
 F 3 "~" H 1250 850 50  0001 C CNN
 	1    1250 850
@@
 F 0 "SW1" H 900 1135 50  0000 C CNN
 F 1 "RESET" H 900 1044 50  0000 C CNN
-F 2 "" H 900 1050 50  0001 C CNN
+F 2 "Button_Switch_THT:KSA_Tactile_SPST" H 900 1050 50  0001 C CNN
 F 3 "~" H 900 1050 50  0001 C CNN
 	1    900  850
@@
 F 0 "C1" V 1050 1000 50  0000 C CNN
 F 1 "100n" V 1150 1000 50  0000 C CNN
-F 2 "" H 938 850 50  0001 C CNN
+F 2 "Capacitor_THT:C_Rect_L10.0mm_W5.0mm_P5.00mm_P7.50mm" H 938 850 50  0001 C CNN
 F 3 "~" H 900 1000 50  0001 C CNN
 	1    900  1000
@@
 F 0 "D1" V 2450 4850 50  0000 R CNN
 F 1 "1N4148" V 2350 4950 50  0000 R CNN
-F 2 "" H 2450 4600 50  0001 C CNN
+F 2 "Diode_THT:D_DO-34_SOD68_P2.54mm_Vertical_AnodeUp" H 2450 4600 50  0001 C CNN
 F 3 "~" H 2450 4600 50  0001 C CNN
 	1    2450 4600
@@
 F 0 "J3" H 7930 3642 50  0000 L CNN
 F 1 "IO8 PORT" H 7930 3551 50  0000 L CNN
-F 2 "" H 7850 3600 50  0001 C CNN
+F 2 "Connector_PinHeader_2.54mm:PinHeader_1x13_P2.54mm_Vertical" H 7850 3600 50  0001 C CNN
 F 3 "~" H 7850 3600 50  0001 C CNN
 	1    7850 3600
@@
 F 0 "J2" H 8730 5242 50  0000 L CNN
 F 1 "IO9 INPUT" H 8730 5151 50  0000 L CNN
-F 2 "" H 8650 5250 50  0001 C CNN
+F 2 "Connector_PinHeader_2.54mm:PinHeader_1x10_P2.54mm_Vertical" H 8650 5250 50  0001 C CNN
 F 3 "~" H 8650 5250 50  0001 C CNN
 	1    8650 5250
@@
 F 0 "BZ1" H 8202 1829 50  0000 L CNN
 F 1 "Buzzer" H 8202 1738 50  0000 L CNN
-F 2 "" V 8025 1900 50  0001 C CNN
+F 2 "Buzzer_Beeper:Buzzer_12x9.5RM7.6" V 8025 1900 50  0001 C CNN
 F 3 "~" V 8025 1900 50  0001 C CNN
 	1    8050 1800
@@
 F 0 "R5" V 7900 1950 50  0000 C CNN
 F 1 "22" V 7900 1800 50  0000 C CNN
-F 2 "" V 7730 1900 50  0001 C CNN
+F 2 "Resistor_THT:R_Axial_DIN0204_L3.6mm_D1.6mm_P2.54mm_Vertical" V 7730 1900 50  0001 C CNN
 F 3 "~" H 7800 1900 50  0001 C CNN
 	1    7800 1900
@@
 Text Label 8350 5450 0    50   ~ 0
 DI1
-Wire Bus Line
-	3200 750  3200 2550
 $Comp
 L Display_Character:LTC4622G U12
@@
 F 0 "U12" H 2375 6767 50  0000 C CNN
 F 1 "LTC4622G" H 2375 6676 50  0000 C CNN
-F 2 "" H 1550 5400 50  0001 L CNN
+F 2 "Connector_PinHeader_2.54mm:PinHeader_1x09_P2.54mm_Vertical" H 1550 5400 50  0001 L CNN
 F 3 "" H 2160 6440 50  0001 L CNN
 	1    2050 6100
@@
 Wire Bus Line
 	4650 1050 4650 6500
+Wire Bus Line
+	3200 750  3200 2550
 $EndSCHEMATC
