File: hard/kicad/iox-kbd/iox-kbd.kicad_pcb (KiCad board)
At the start: 2 copper layers, 14 parts, among them J1 IOX, J2 VIAport2, U1 74HC132, U2 27C512, U3 27C512, U4 74HC174, U5 74HC4024

Commit message: work on Durango-X np board
Routing:
- net +5V: track 130.5 -> 228.4 mm, vias 1 -> 4
- net GND: track 159.8 -> 254.3 mm, vias 2 -> 3
- net /~MOD: track 2.54 -> 87.4 mm, vias 0 -> 2
- net /~CAPSLOCK: track 21.3 -> 104.1 mm, vias 0 -> 2
- net Net-(C2-Pad1): track 0.00 -> 80.3 mm, vias 0 -> 2
- net Net-(C1-Pad2): track 0.00 -> 71.9 mm, vias 0 -> 2
- net Net-(U1-Pad11): track 0.00 -> 68.4 mm, vias 0 -> 1
- net /~WE: track 0.00 -> 67.3 mm, vias 0 -> 1
- net Net-(R1-Pad1): track 21.9 -> 81.1 mm, vias 0 -> 1
- net /~SEL: track 2.54 -> 58.0 mm, vias 0 -> 1
- net /CTL: track 0.00 -> 47.0 mm, vias 0 -> 1
- net Net-(U2-Pad24): track 21.3 -> 61.9 mm, vias 0 -> 1
- net /~CAPS: track 0.00 -> 40.2 mm, vias 0 -> 2
- net /SHIFT: track 0.00 -> 39.9 mm, vias 0 -> 1
- net /D7: track 5.08 -> 44.3 mm, vias 0 -> 2
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