File: hard/kicad/debug/debug.kicad_pcb (KiCad board)
At the start: 2 copper layers, 6 parts, among them J1 6502 DEBUG, U1 74HC374, U2 74HC139, U3 LTC4622G

Commit message: improvements in GBA POC Pacman
Routing:
- net +5V: track 36.9 -> 17.6 mm
- net GND: track 66.0 -> 55.2 mm
- added copper zone on B.Cu, net +5V
- added copper zone on F.Cu, net GND
Other:
- board outline added: 42.5 x 44.5 mm
Changed lines of the file:
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@@
   (general
     (thickness 1.6)
-    (drawings 2)
-    (tracks 185)
+    (drawings 6)
+    (tracks 178)
     (zones 0)
     (modules 6)
@@
     )
   )
+  (gr_line (start 20.955 15.875) (end 20.955 60.325) (layer Edge.Cuts) (width 0.0254))
+  (gr_line (start 63.5 15.875) (end 20.955 15.875) (layer Edge.Cuts) (width 0.0254))
+  (gr_line (start 63.5 60.325) (end 63.5 15.875) (layer Edge.Cuts) (width 0.0254))
+  (gr_line (start 20.955 60.325) (end 63.5 60.325) (layer Edge.Cuts) (width 0.0254))
   (gr_text JLCJLCJLCJLC (at 53.34 20.574) (layer B.SilkS)
     (effects (font (size 1.5 1.5) (thickness 0.3)) (justify mirror))
@@
     (effects (font (size 1.5 1.5) (thickness 0.3)))
   )
-  (segment (start 38.1 20.4) (end 41.736 20.4) (width 1) (layer F.Cu) (net 1))
   (segment (start 43.18 21.844) (end 43.18 30.48) (width 1) (layer F.Cu) (net 1))
   (segment (start 41.736 20.4) (end 43.18 21.844) (width 1) (layer F.Cu) (net 1))
-  (segment (start 45.72 50.8) (end 43.18 53.34) (width 1) (layer F.Cu) (net 1))
   (segment (start 45.72 33.02) (end 45.72 50.8) (width 1) (layer F.Cu) (net 1))
-  (segment (start 43.18 30.48) (end 45.72 33.02) (width 1) (layer F.Cu) (net 1))
   (segment (start 43.18 53.34) (end 33.02 53.34) (width 1) (layer B.Cu) (net 1))
   (segment (start 33.02 53.34) (end 27.94 58.42) (width 1) (layer B.Cu) (net 1))
@@
   (segment (start 31.75 48.26) (end 33.02 49.53) (width 0.254) (layer F.Cu) (net 1))
   (segment (start 33.02 49.53) (end 33.02 53.34) (width 0.254) (layer F.Cu) (net 1))
-  (segment (start 38.1 25.4) (end 48.26 25.4) (width 1) (layer B.Cu) (net 2))
   (segment (start 48.26 25.4) (end 50.8 27.94) (width 1) (layer B.Cu) (net 2))
-  (segment (start 50.8 27.94) (end 50.8 30.48) (width 1) (layer B.Cu) (net 2))
   (segment (start 38.1 25.4) (end 38.1 30.48) (width 0.254) (layer F.Cu) (net 2))
   (segment (start 34.29 20.32) (end 25.4 20.32) (width 1) (layer B.Cu) (net 2))
-  (segment (start 38.1 24.13) (end 34.29 20.32) (width 1) (layer B.Cu) (net 2))
-  (segment (start 38.1 25.4) (end 38.1 24.13) (width 1) (layer B.Cu) (net 2))
   (segment (start 25.4 53.34) (end 27.432 53.34) (width 0.127) (layer F.Cu) (net 3))
   (segment (start 27.432 53.34) (end 28.194 52.578) (width 0.127) (layer F.Cu) (net 3))
@@
   (segment (start 44.659736 41.148) (end 48.26 41.148) (width 0.127) (layer B.Cu) (net 7))
   (segment (start 48.26 41.148) (end 48.26 41.148) (width 0.127) (layer B.Cu) (net 7))
-  (via (at 48.26 41.148) (size 0.6) (drill 0.3) (layers F.Cu B.Cu) (net 7) (status 1000000))
+  (via (at 48.26 41.148) (size 0.6) (drill 0.3) (layers F.Cu B.Cu) (net 7))
   (segment (start 48.26 41.148) (end 48.26 40.64) (width 0.127) (layer F.Cu) (net 7))
   (segment (start 48.26 40.64) (end 50.8 38.1) (width 0.127) (layer F.Cu) (net 7))
@@
   (segment (start 34.798 46.99) (end 36.068 48.26) (width 0.127) (layer F.Cu) (net 29))
   (segment (start 36.068 48.26) (end 38.1 48.26) (width 0.127) (layer F.Cu) (net 29))
+  (zone (net 2) (net_name +5V) (layer B.Cu) (hatch edge 0.508)
+    (connect_pads (clearance 0.508))
+    (min_thickness 0.254)
+    (fill yes (arc_segments 32) (thermal_gap 0.508) (thermal_bridge_width 0.508))
+    (polygon
+      (pts
+        (xy 20.32 60.96) (xy 20.32 15.24) (xy 64.77 15.24) (xy 64.135 60.96)
+      )
+    )
+  )
+  (zone (net 1) (net_name GND) (layer F.Cu) (hatch edge 0.508)
+    (connect_pads (clearance 0.508))
+    (min_thickness 0.254)
+    (fill yes (arc_segments 32) (thermal_gap 0.508) (thermal_bridge_width 0.508))
+    (polygon
+      (pts
+        (xy 20.32 60.96) (xy 20.32 15.24) (xy 64.135 15.24) (xy 64.135 60.96)
+      )
+    )
+  )
 )

Commit message: fixes on 6502debug PCB
Parts:
- added JP1: +5V, Connector_PinHeader_2.54mm:PinHeader_1x02_P2.54mm_Vertical, F.Cu at (30.5, 22.9)
Connections:
- J1 pad 16: +5V -> /VDD
Routing:
- net +5V: track 17.6 -> 5.08 mm
- net /VDD: track 0.00 -> 5.08 mm
Changed lines of the file:
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@@
     (thickness 1.6)
     (drawings 6)
-    (tracks 178)
+    (tracks 177)
     (zones 0)
-    (modules 6)
-    (nets 30)
+    (modules 7)
+    (nets 31)
   )
   (page A4)
@@
   )
   (setup
-    (last_trace_width 0.25)
+    (last_trace_width 1)
     (user_trace_width 0.127)
     (user_trace_width 0.1778)
@@
       (outputformat 1)
       (mirror false)
-      (drillshape 1)
+      (drillshape 0)
       (scaleselection 1)
       (outputdirectory ""))
@@
   (net 28 /~DISP)
   (net 29 /~ROM)
+  (net 30 /VDD)
   (net_class Default "Esta es la clase de red por defecto."
     (clearance 0.2)
@@
     (add_net /KPG)
     (add_net /R~W)
+    (add_net /VDD)
     (add_net /~DISP)
     (add_net /~ROM)
@@
     (uvia_drill 0.2)
   )
+  (module Connector_PinHeader_2.54mm:PinHeader_1x02_P2.54mm_Vertical (layer F.Cu)
+    (at 30.48 22.86 180)
+    (descr "Through hole straight pin header, 1x02, 2.54mm pitch, single row")
+    (tags "Through hole pin header THT 1x02 2.54mm single row")
+    (fp_text reference JP1 (at -2.54 1.27 270 unlocked) (layer B.SilkS)
+      (effects (font (size 1 1) (thickness 0.15)) (justify mirror))
+    )
+    (fp_text value +5V (at 0 -3.175 270 unlocked) (layer F.SilkS)
+      (effects (font (size 1 1) (thickness 0.15)))
+    )
+    (fp_text user %R (at 0 1.27 90) (layer F.Fab)
+      (effects (font (size 1 1) (thickness 0.15)))
+    )
+    (fp_line (start 1.8 -1.8) (end -1.8 -1.8) (layer F.CrtYd) (width 0.05))
+    (fp_line (start 1.8 4.35) (end 1.8 -1.8) (layer F.CrtYd) (width 0.05))
+    (fp_line (start -1.8 4.35) (end 1.8 4.35) (layer F.CrtYd) (width 0.05))
+    (fp_line (start -1.8 -1.8) (end -1.8 4.35) (layer F.CrtYd) (width 0.05))
+    (fp_line (start -1.33 -1.33) (end 0 -1.33) (layer F.SilkS) (width 0.12))
+    (fp_line (start -1.33 0) (end -1.33 -1.33) (layer F.SilkS) (width 0.12))
+    (fp_line (start -1.33 1.27) (end 1.33 1.27) (layer F.SilkS) (width 0.12))
+    (fp_line (start 1.33 1.27) (end 1.33 3.87) (layer F.SilkS) (width 0.12))
+    (fp_line (start -1.33 1.27) (end -1.33 3.87) (layer F.SilkS) (width 0.12))
+    (fp_line (start -1.33 3.87) (end 1.33 3.87) (layer F.SilkS) (width 0.12))
+    (fp_line (start -1.27 -0.635) (end -0.635 -1.27) (layer F.Fab) (width 0.1))
+    (fp_line (start -1.27 3.81) (end -1.27 -0.635) (layer F.Fab) (width 0.1))
+    (fp_line (start 1.27 3.81) (end -1.27 3.81) (layer F.Fab) (width 0.1))
+    (fp_line (start 1.27 -1.27) (end 1.27 3.81) (layer F.Fab) (width 0.1))
+    (fp_line (start -0.635 -1.27) (end 1.27 -1.27) (layer F.Fab) (width 0.1))
+    (pad 2 thru_hole oval (at 0 2.54 180) (size 1.7 1.7) (drill 1) (layers *.Cu *.Mask)
+      (net 30 /VDD))
+    (pad 1 thru_hole rect (at 0 0 180) (size 1.7 1.7) (drill 1) (layers *.Cu *.Mask)
+      (net 2 +5V))
+    (model ${KISYS3DMOD}/Connector_PinHeader_2.54mm.3dshapes/PinHeader_1x02_P2.54mm_Vertical.wrl
+      (at (xyz 0 0 0))
+      (scale (xyz 1 1 1))
+      (rotate (xyz 0 0 0))
+    )
+  )
   (module Connector_PinSocket_2.54mm:PinSocket_1x09_P2.54mm_Vertical (layer F.Cu)
     (at 60.96 27.94)
@@
       (effects (font (size 1 1) (thickness 0.15)) (justify mirror))
     )
-    (fp_text value LTC4622G (at -2.54 2.032 270 unlocked) (layer F.SilkS)
+    (fp_text value LTC4622G (at 0 26.035 270 unlocked) (layer F.SilkS)
       (effects (font (size 1 1) (thickness 0.15)))
     )
@@
       (effects (font (size 1 1) (thickness 0.15)) (justify mirror))
     )
-    (fp_text value "6502 DEBUG" (at -2.794 36.576 270 unlocked) (layer F.SilkS)
-      (effects (font (size 1 1) (thickness 0.15)))
-    )
-    (fp_text user %R (at 2.77 20.32 90) (layer F.Fab)
+    (fp_text value "6502 DEBUG" (at -5.08 3.175 270 unlocked) (layer F.SilkS)
       (effects (font (size 1 1) (thickness 0.15)))
     )
@@
       (net 15 /CLK))
     (pad 16 thru_hole oval (at 0 38.1 180) (size 1.7 1.7) (drill 1) (layers *.Cu *.Mask)
-      (net 2 +5V))
+      (net 30 /VDD))
     (pad 15 thru_hole oval (at 0 35.56 180) (size 1.7 1.7) (drill 1) (layers *.Cu *.Mask))
     (pad 14 thru_hole oval (at 0 33.02 180) (size 1.7 1.7) (drill 1) (layers *.Cu *.Mask)
@@
   (gr_line (start 63.5 60.325) (end 63.5 15.875) (layer Edge.Cuts) (width 0.0254))
   (gr_line (start 20.955 60.325) (end 63.5 60.325) (layer Edge.Cuts) (width 0.0254))
-  (gr_text JLCJLCJLCJLC (at 53.34 20.574) (layer B.SilkS)
+  (gr_text JLCJLCJLCJLC (at 54.61 17.78) (layer B.SilkS)
     (effects (font (size 1.5 1.5) (thickness 0.3)) (justify mirror))
   )
@@
   (segment (start 31.75 48.26) (end 33.02 49.53) (width 0.254) (layer F.Cu) (net 1))
   (segment (start 33.02 49.53) (end 33.02 53.34) (width 0.254) (layer F.Cu) (net 1))
-  (segment (start 48.26 25.4) (end 50.8 27.94) (width 1) (layer B.Cu) (net 2))
   (segment (start 38.1 25.4) (end 38.1 30.48) (width 0.254) (layer F.Cu) (net 2))
-  (segment (start 34.29 20.32) (end 25.4 20.32) (width 1) (layer B.Cu) (net 2))
   (segment (start 25.4 53.34) (end 27.432 53.34) (width 0.127) (layer F.Cu) (net 3))
   (segment (start 27.432 53.34) (end 28.194 52.578) (width 0.127) (layer F.Cu) (net 3))
@@
   (segment (start 34.798 46.99) (end 36.068 48.26) (width 0.127) (layer F.Cu) (net 29))
   (segment (start 36.068 48.26) (end 38.1 48.26) (width 0.127) (layer F.Cu) (net 29))
+  (segment (start 25.4 20.32) (end 30.48 20.32) (width 1) (layer B.Cu) (net 30))
   (zone (net 2) (net_name +5V) (layer B.Cu) (hatch edge 0.508)
     (connect_pads (clearance 0.508))
