File: hard/kicad/debug/debug.sch (KiCad schematic (older format))
At the start: 6 parts, among them J1 6502 DEBUG, U1 74HC374, U2 74HC139, U3 LTC4622G

Commit message: fixes on 6502debug PCB
Parts:
- added JP1: +5V, Connector_PinHeader_2.54mm:PinHeader_1x02_P2.54mm_Vertical, symbol Device:Jumper_NC_Small
Connections:
- net +5V: now also JP1.1; no longer J1.16 (Pin_16)
- new net VDD: J1.16 (Pin_16), JP1.2
Changed lines of the file:
@@
 Wire Wire Line
 	2750 3800 2750 5000
-Wire Wire Line
-	1150 5000 1150 3500
 $Comp
 L power:+5V #PWR0102
@@
 	0    1    1    0
 $EndComp
-Connection ~ 1150 3500
 Wire Wire Line
 	1150 3500 1150 3300
@@
 	1    0    0    -1
 $EndComp
+$Comp
+L Device:Jumper_NC_Small JP1
+U 1 1 61A58ADE
+P 1150 4700
+F 0 "JP1" V 1104 4774 50  0000 L CNN
+F 1 "+5V" V 1195 4774 50  0000 L CNN
+F 2 "Connector_PinHeader_2.54mm:PinHeader_1x02_P2.54mm_Vertical" H 1150 4700 50  0001 C CNN
+F 3 "~" H 1150 4700 50  0001 C CNN
+	1    1150 4700
+	0    1    1    0
+$EndComp
+Wire Wire Line
+	1150 4800 1150 5000
+Wire Wire Line
+	1150 4600 1150 3500
+Connection ~ 1150 3500
 $EndSCHEMATC
