File: hard/kicad/durango/rgb-test/rgb-test.kicad_pcb (KiCad board)
At the start: 2 copper layers, 23 parts, among them J1 SCART, J2 POWER, SW1 TEST, U1 74HCT4040, U2 74HC4040, U3 74HC21, U4 74HC02, U5 74HC245, U6 74HC86, U7 74HC85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

Commit message: fill SCART tester
Routing:
- added copper zone on B.Cu, net +5V
- added copper zone on F.Cu, net GND
Changed lines of the file:
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@@
     (add_net /~VS)
     (add_net GND)
-    (add_net "Net-(J1-Pad1)")
-    (add_net "Net-(J1-Pad10)")
-    (add_net "Net-(J1-Pad12)")
-    (add_net "Net-(J1-Pad14)")
-    (add_net "Net-(J1-Pad17)")
-    (add_net "Net-(J1-Pad19)")
-    (add_net "Net-(J1-Pad3)")
-    (add_net "Net-(J2-Pad2)")
-    (add_net "Net-(J2-Pad3)")
     (add_net "Net-(R5-Pad2)")
-    (add_net "Net-(U1-Pad1)")
     (add_net "Net-(U1-Pad10)")
-    (add_net "Net-(U1-Pad3)")
-    (add_net "Net-(U1-Pad4)")
-    (add_net "Net-(U1-Pad5)")
-    (add_net "Net-(U1-Pad6)")
-    (add_net "Net-(U1-Pad7)")
-    (add_net "Net-(U1-Pad9)")
-    (add_net "Net-(U2-Pad1)")
-    (add_net "Net-(U2-Pad14)")
-    (add_net "Net-(U2-Pad15)")
     (add_net "Net-(U2-Pad3)")
     (add_net "Net-(U2-Pad5)")
     (add_net "Net-(U2-Pad6)")
-    (add_net "Net-(U2-Pad7)")
-    (add_net "Net-(U2-Pad9)")
-    (add_net "Net-(U5-Pad8)")
-    (add_net "Net-(U5-Pad9)")
-    (add_net "Net-(U7-Pad5)")
-    (add_net "Net-(U7-Pad7)")
-    (add_net "Net-(U8-Pad5)")
-    (add_net "Net-(U8-Pad7)")
-    (add_net "Net-(X1-Pad1)")
   )
   (module Package_DIP:DIP-14_W7.62mm_Socket (layer F.Cu)
@@
   (segment (start 68.449997 48.390003) (end 69.85 46.99) (width 0.25) (layer F.Cu) (net 37))
   (segment (start 68.449997 54.61) (end 68.449997 48.390003) (width 0.25) (layer F.Cu) (net 37))
+  (zone (net 3) (net_name GND) (layer F.Cu) (hatch edge 0.508)
+    (connect_pads (clearance 0.508))
+    (min_thickness 0.254)
+    (fill yes (arc_segments 32) (thermal_gap 0.508) (thermal_bridge_width 0.508))
+    (polygon
+      (pts
+        (xy 31.115 85.09) (xy 31.115 31.75) (xy 104.775 31.75) (xy 104.775 85.09)
+      )
+    )
+  )
+  (zone (net 7) (net_name +5V) (layer B.Cu) (hatch edge 0.508)
+    (connect_pads (clearance 0.508))
+    (min_thickness 0.254)
+    (fill yes (arc_segments 32) (thermal_gap 0.508) (thermal_bridge_width 0.508))
+    (polygon
+      (pts
+        (xy 31.115 31.75) (xy 104.775 31.75) (xy 104.775 85.09) (xy 31.115 85.09)
+      )
+    )
+  )
 )
