File: hard/kicad/pendrive/pendrive.sch (KiCad schematic (older format))
At the start: 8 parts, among them J1 IOx, U1 62256, U2 74HC138, U3 74HC574, U4 74HC574

Commit message: retraced pendrive
Parts:
- added LOGO1: Logo_Open_Hardware_Small, durango:jaqueria, symbol Graphic:Logo_Open_Hardware_Small
- added LOGO2: Logo_Open_Hardware_Large, Symbol:OSHW-Logo_19x20mm_SilkScreen, symbol Graphic:Logo_Open_Hardware_Large
- D1: value D_Schottky -> BAT43
Connections:
- net A0: now also U1.3 (A7); no longer U1.10 (A0)
- net A1: now also U1.4 (A6); no longer U1.9 (A1)
- net A10: now also U1.25 (A8); no longer U1.24 (A9)
- net A11: now also U1.24 (A9); no longer U1.25 (A8)
- net A12: now also U1.23 (A11); no longer U1.26 (A13)
- net A13: now also U1.21 (A10); no longer U1.2 (A12)
- net A2: now also U1.5 (A5); no longer U1.8 (A2)
- net A3: now also U1.6 (A4); no longer U1.7 (A3)
- net A4: now also U1.7 (A3); no longer U1.6 (A4)
- net A5: now also U1.8 (A2); no longer U1.5 (A5)
- net A6: now also U1.9 (A1); no longer U1.4 (A6)
- net A7: now also U1.10 (A0); no longer U1.3 (A7)
- net A8: now also U1.2 (A12); no longer U1.21 (A10)
- net A9: now also U1.26 (A13); no longer U1.23 (A11)
- net PD0: now also U1.19 (D7); no longer U1.13 (D2)
- net PD1: now also U1.18 (D6); no longer U1.12 (D1)
- net PD3: now also U1.17 (D5); no longer U1.15 (D3)
- net PD4: now also U1.12 (D1); no longer U1.16 (D4)
- net PD5: now also U1.16 (D4); no longer U1.17 (D5)
- net PD6: now also U1.13 (D2); no longer U1.18 (D6)
- net PD7: now also U1.15 (D3); no longer U1.19 (D7)
Changed lines of the file:
@@
 P 5350 2750
 F 0 "D1" H 5350 2850 50  0000 C CNN
-F 1 "D_Schottky" H 5425 2650 50  0000 C CNN
+F 1 "BAT43" H 5350 2650 50  0000 C CNN
 F 2 "Diode_THT:D_DO-35_SOD27_P10.16mm_Horizontal" H 5350 2750 50  0001 C CNN
 F 3 "~" H 5350 2750 50  0001 C CNN
@@
 Text Label 4100 5000 0    50   ~ 0
 A8
-Text Label 4550 4150 2    50   ~ 0
+Text Label 4600 4150 2    50   ~ 0
+A12
+Text Label 4600 3950 2    50   ~ 0
+A11
+Text Label 4600 3850 2    50   ~ 0
+A10
+Text Label 4550 4350 2    50   ~ 0
 A9
-Text Label 4600 3950 2    50   ~ 0
-A10
-Text Label 4600 3850 2    50   ~ 0
-A11
-Text Label 4600 4350 2    50   ~ 0
-A12
-Text Label 4600 4250 2    50   ~ 0
-A13
+Text Label 4550 4250 2    50   ~ 0
+A8
 Text Label 4600 4450 2    50   ~ 0
 A14
@@
 PD2
 Text Label 5800 3150 0    50   ~ 0
+PD4
+Text Label 5800 3250 0    50   ~ 0
+PD6
+Text Label 5800 3350 0    50   ~ 0
+PD7
+Text Label 5800 3450 0    50   ~ 0
+PD5
+Text Label 5800 3550 0    50   ~ 0
+PD3
+Text Label 5800 3650 0    50   ~ 0
 PD1
-Text Label 5800 3250 0    50   ~ 0
+Text Label 5800 3750 0    50   ~ 0
 PD0
-Text Label 5800 3350 0    50   ~ 0
-PD3
-Text Label 5800 3450 0    50   ~ 0
-PD4
-Text Label 5800 3550 0    50   ~ 0
-PD5
-Text Label 5800 3650 0    50   ~ 0
-PD6
-Text Label 5800 3750 0    50   ~ 0
-PD7
 Text Label 4100 2500 0    50   ~ 0
 PD[0..7]
@@
 	4450 3750 4600 3750
 Text Label 4450 3050 0    50   ~ 0
+A7
+Text Label 4450 3150 0    50   ~ 0
+A6
+Text Label 4450 3250 0    50   ~ 0
+A5
+Text Label 4450 3350 0    50   ~ 0
+A4
+Text Label 4450 3450 0    50   ~ 0
+A3
+Text Label 4450 3550 0    50   ~ 0
+A2
+Text Label 4450 3650 0    50   ~ 0
+A1
+Text Label 4450 3750 0    50   ~ 0
 A0
-Text Label 4450 3150 0    50   ~ 0
-A1
-Text Label 4450 3250 0    50   ~ 0
-A2
-Text Label 4450 3350 0    50   ~ 0
-A3
-Text Label 4450 3450 0    50   ~ 0
-A4
-Text Label 4450 3550 0    50   ~ 0
-A5
-Text Label 4450 3650 0    50   ~ 0
-A6
-Text Label 4450 3750 0    50   ~ 0
-A7
 Entry Wire Line
 	4250 3050 4350 3150
@@
 	4450 3950 4600 3950
 Text Label 4450 4050 0    50   ~ 0
-A8
+A13
 Entry Wire Line
 	4350 3950 4450 3850
@@
 Wire Wire Line
 	1800 3450 2100 3450
+$Comp
+L Graphic:Logo_Open_Hardware_Small LOGO1
+U 1 1 644B7759
+P 7150 2650
+F 0 "LOGO1" H 7150 2925 50  0001 C CNN
+F 1 "Logo_Open_Hardware_Small" H 7150 2425 50  0001 C CNN
+F 2 "durango:jaqueria" H 7150 2650 50  0001 C CNN
+F 3 "~" H 7150 2650 50  0001 C CNN
+	1    7150 2650
+	1    0    0    -1
+$EndComp
 Wire Bus Line
 	6050 2500 6050 3650
@@
 Wire Bus Line
 	4350 3150 4350 5500
+$Comp
+L Graphic:Logo_Open_Hardware_Large LOGO2
+U 1 1 644DA0AF
+P 7150 3500
+F 0 "LOGO2" H 7150 4000 50  0001 C CNN
+F 1 "Logo_Open_Hardware_Large" H 7150 3100 50  0001 C CNN
+F 2 "Symbol:OSHW-Logo_19x20mm_SilkScreen" H 7150 3500 50  0001 C CNN
+F 3 "~" H 7150 3500 50  0001 C CNN
+	1    7150 3500
+	1    0    0    -1
+$EndComp
 $EndSCHEMATC
