File: hard/kicad/durango/cartridges/cart32bbs/cart32bbs.sch (KiCad schematic (older format))
At the start: 4 parts, among them J1 Durango_ROM, U1 27C010, U2 74HC174, U3 74HC138

Commit message: complete 128K BBS silkscreen
Parts:
- added LOGO1: Logo_Open_Hardware_Small, durango:jaqueria, symbol Graphic:Logo_Open_Hardware_Small
Changed lines of the file:
@@
 EESchema Schematic File Version 4
+LIBS:cart32bbs-cache
 EELAYER 29 0
 EELAYER END
@@
 Wire Bus Line
 	1600 950  1600 4100
+$Comp
+L Graphic:Logo_Open_Hardware_Small LOGO1
+U 1 1 6483E578
+P 6900 1650
+F 0 "LOGO1" H 6900 1925 50  0001 C CNN
+F 1 "Logo_Open_Hardware_Small" H 6900 1425 50  0001 C CNN
+F 2 "durango:jaqueria" H 6900 1650 50  0001 C CNN
+F 3 "~" H 6900 1650 50  0001 C CNN
+	1    6900 1650
+	1    0    0    -1
+$EndComp
 $EndSCHEMATC

Commit message: update BBS cartridge
Parts:
- removed U1: 27C010, Package_DIP:DIP-32_W15.24mm, symbol Memory_EPROM:27C010
- added JP1: 16/32K, Jumper:SolderJumper-3_P1.3mm_Bridged12_RoundedPad1.0x1.5mm, symbol Jumper:Jumper_3_Bridged12
- added JP2: 040+, Jumper:SolderJumper-3_P1.3mm_Bridged12_RoundedPad1.0x1.5mm, symbol Jumper:Jumper_3_Bridged12
- added JP3: 080, Jumper:SolderJumper-3_P1.3mm_Bridged12_RoundedPad1.0x1.5mm, symbol Jumper:Jumper_3_Bridged12
- added U1: 27C010-080, Package_DIP:DIP-32_W15.24mm, symbol Memory_EPROM:27C080
Connections:
- net +5V: now also JP2.1 (A), JP3.1 (A), U1.32 (VCC); no longer U2.11 (D3), U2.13 (D4), U2.14 (D5)
- net A0: now also U1.12 (A0)
- net A1: now also U1.11 (A1)
- net A10: now also U1.23 (A10)
- net A11: now also U1.25 (A11)
- net A12: now also U1.4 (A12)
- net A13: now also U1.28 (A13)
- net A2: now also U1.10 (A2)
- net A3: now also U1.9 (A3)
- net A4: now also U1.8 (A4)
- net A5: now also U1.7 (A5)
- net A6: now also U1.6 (A6)
- net A7: now also U1.5 (A7)
- net A8: now also U1.27 (A8)
- net A9: now also U1.26 (A9)
- net BA0: now also JP1.3 (B)
- net BA1: now also U1.3 (A15)
- net BA2: now also U1.2 (A16)
- net D0: now also U1.13 (D0)
- net D1: now also U1.14 (D1)
- net D2: now also U1.15 (D2)
- net D3: now also U2.11 (D3), U1.17 (D3)
- net D4: now also U2.13 (D4), U1.18 (D4)
- net D5: now also U2.14 (D5), U1.19 (D5)
- net D6: now also U1.20 (D6)
- net D7: now also U1.21 (D7)
- net GND: now also U1.16 (GND)
- net ~CS: now also U1.22 (~CE)
- net ~OE: now also U1.24 (~OE)
- net A14: now reaches J1.9 (A14)
- net A14: now also JP1.1 (A)
- net BA3: now reaches U2.10 (Q3)
- net BA3: now also U1.30 (A17)
- net BA4: now reaches U2.12 (Q4)
- net BA4: now also JP2.3 (B)
- net BA5: now reaches U2.15 (Q5)
- net BA5: now also JP3.3 (B)
- new net MA14: JP1.2 (C), U1.29 (A14)
- new net MA18: JP2.2 (C), U1.31 (A18)
- new net MA19: JP3.2 (C), U1.1 (A19)
- no-connect marks 15 -> 11
Other:
- note added: "8/16/32/64x 16 KiB\n4/8/16/32x 32 KiB\nI/O = $DFFC-DFFF"
- note removed: "8x 16 KiB\nI/O = $DFF0-DFF3"
Changed lines of the file:
@@
-$EndComp
-$Comp
-L Memory_EPROM:27C010 U1
-U 1 1 6482130A
-P 5500 2550
-F 0 "U1" H 5250 3700 50  0000 C CNN
-F 1 "27C010" H 5700 3700 50  0000 C CNN
-F 2 "Package_DIP:DIP-32_W15.24mm" H 5500 2550 50  0001 C CNN
-F 3 "http://ww1.microchip.com/downloads/en/DeviceDoc/doc0321.pdf" H 5500 2550 50  0001 C CNN
-	1    5500 2550
-	1    0    0    -1
 $EndComp
 $Comp
@@
 	1    0    0    -1
 $EndComp
-Text Notes 3550 850  0    100  ~ 20
-8x 16 KiB\nI/O = $DFF0-DFF3
+Text Notes 6100 3050 0    100  ~ 0
+8/16/32/64x 16 KiB\n4/8/16/32x 32 KiB\nI/O = $DFFC-DFFF
 $Comp
 L power:GND #PWR0101
@@
 Wire Wire Line
 	3900 4700 5500 4700
-Wire Wire Line
-	5500 4700 5500 3850
 Connection ~ 3900 4700
 Text Label 1900 1350 2    50   ~ 0
@@
 	1    0    0    -1
 $EndComp
-Connection ~ 3900 3400
 $Comp
 L power:GND #PWR0104
@@
 $EndComp
 NoConn ~ 2750 1350
-Wire Wire Line
-	5100 3450 5100 3400
-Wire Wire Line
-	3900 3400 5100 3400
-Connection ~ 5100 3400
-Wire Wire Line
-	5100 3400 5100 3350
 NoConn ~ 2750 2750
 NoConn ~ 2750 2850
 NoConn ~ 2750 3050
 Wire Wire Line
-	2750 2550 3100 2550
-Wire Wire Line
-	3100 2550 3100 3150
-Wire Wire Line
-	3100 3150 4550 3150
-Wire Wire Line
-	4550 3150 4550 3550
-Wire Wire Line
-	4550 3550 5100 3550
-Wire Wire Line
-	2750 2450 3150 2450
-Wire Wire Line
-	3150 2450 3150 3100
-Wire Wire Line
-	3150 3100 4500 3100
-Wire Wire Line
-	4500 3100 4500 3650
-Wire Wire Line
-	4500 3650 5100 3650
-Text Label 4550 3550 0    50   ~ 0
+	2750 2550 2800 2550
+Wire Wire Line
+	2800 2550 2800 5100
+Wire Wire Line
+	2750 2450 2850 2450
+Wire Wire Line
+	2850 2450 2850 5000
+Text Label 4650 5100 0    50   ~ 0
 ~CS
-Text Label 4500 3650 0    50   ~ 0
+Text Label 4950 5000 0    50   ~ 0
 ~OE
 Wire Wire Line
@@
 Wire Wire Line
 	1700 2850 1950 2850
-NoConn ~ 1950 2950
 Text Label 1750 1550 0    50   ~ 0
 A0
@@
 	4750 950  1600 950
 Text GLabel 1600 950  0    50   Input ~ 0
-A[0..13]
+A[0..14]
 Text GLabel 6250 1000 2    50   Input ~ 0
 D[0..7]
 Text Label 5100 2950 2    50   ~ 0
+MA14
+Text Label 5050 3050 2    50   ~ 0
+BA1
+Text Label 5050 3150 2    50   ~ 0
+BA2
+Entry Wire Line
+	3050 1450 3150 1550
+Entry Wire Line
+	3050 1550 3150 1650
+Entry Wire Line
+	3050 1650 3150 1750
+Wire Wire Line
+	3150 1550 3400 1550
+Wire Wire Line
+	3150 1650 3400 1650
+Wire Wire Line
+	3150 1750 3400 1750
+Text Label 3200 1650 0    50   ~ 0
+D1
+Text Label 3200 1750 0    50   ~ 0
+D2
+Text Label 4400 1550 0    50   ~ 0
 BA0
-Text Label 5100 3050 2    50   ~ 0
+Text Label 4400 1650 0    50   ~ 0
 BA1
-Text Label 5100 3150 2    50   ~ 0
+Text Label 4400 1750 0    50   ~ 0
 BA2
-Entry Wire Line
-	3050 1450 3150 1550
-Entry Wire Line
-	3050 1550 3150 1650
-Entry Wire Line
-	3050 1650 3150 1750
-Wire Wire Line
-	3150 1550 3400 1550
-Wire Wire Line
-	3150 1650 3400 1650
-Wire Wire Line
-	3150 1750 3400 1750
-Text Label 3200 1650 0    50   Italic 0
-D1
-Text Label 3200 1750 0    50   Italic 0
-D2
-Text Label 4400 1550 0    50   Italic 0
-BA0
-Text Label 4400 1650 0    50   Italic 0
-BA1
-Text Label 4400 1750 0    50   Italic 0
-BA2
-Wire Wire Line
-	4400 1750 4600 1750
-Wire Wire Line
-	4600 1750 4600 3150
-Wire Wire Line
-	4600 3150 5100 3150
-Wire Wire Line
-	4400 1650 4650 1650
-Wire Wire Line
-	4650 1650 4650 3050
-Wire Wire Line
-	4650 3050 5100 3050
-Wire Wire Line
-	4400 1550 4700 1550
-Wire Wire Line
-	4700 1550 4700 2950
-Wire Wire Line
-	4700 2950 5100 2950
-Wire Wire Line
-	3400 1850 3400 1950
-Connection ~ 3400 1950
-Wire Wire Line
-	3400 1950 3400 2050
-$Comp
-L power:+5V #PWR0106
-U 1 1 648631C0
-P 3400 1950
-F 0 "#PWR0106" H 3400 1800 50  0001 C CNN
-F 1 "+5V" V 3415 2078 50  0000 L CIN
-F 2 "" H 3400 1950 50  0001 C CNN
-F 3 "" H 3400 1950 50  0001 C CNN
-	1    3400 1950
-	0    -1   -1   0
-$EndComp
-NoConn ~ 4400 1850
-NoConn ~ 4400 1950
-NoConn ~ 4400 2050
-Text Label 3200 1550 0    50   Italic 0
+Wire Wire Line
+	4400 1750 4650 1750
+Wire Wire Line
+	4650 1750 4650 3150
+Wire Wire Line
+	4650 3150 5100 3150
+Wire Wire Line
+	4400 1650 4700 1650
+Wire Wire Line
+	4700 1650 4700 3050
+Wire Wire Line
+	4700 3050 5100 3050
+Text Label 3200 1550 0    50   ~ 0
 D0
 Wire Wire Line
@@
 Wire Wire Line
 	1900 4300 3400 4300
-Text Label 2650 4300 0    50   Italic 0
+Text Label 3250 4300 0    50   ~ 0
 ~IOC
-Text Label 2650 4400 0    50   Italic 0
+Text Label 3250 4400 0    50   ~ 0
 ~WE
 Entry Wire Line
@@
 Wire Wire Line
 	1700 4200 3400 4200
-Text Label 1750 4200 0    50   Italic 0
+Text Label 1750 4200 0    50   ~ 0
 A5
-Text Label 1750 3900 0    50   Italic 0
+Text Label 1750 3900 0    50   ~ 0
 A4
-Text Label 1750 3800 0    50   Italic 0
+Text Label 1750 3800 0    50   ~ 0
 A3
-Text Label 1750 3700 0    50   Italic 0
+Text Label 1750 3700 0    50   ~ 0
 A2
 NoConn ~ 4400 3700
@@
 Wire Wire Line
 	4400 4950 4400 4400
-Text Label 4400 4500 0    50   Italic 0
+Text Label 4400 4500 0    50   ~ 0
 ~LATCH
 Wire Wire Line
@@
 Wire Wire Line
 	1500 1350 1950 1350
+$Comp
+L Graphic:Logo_Open_Hardware_Small LOGO1
+U 1 1 6483E578
+P 6900 1650
+F 0 "LOGO1" H 6900 1925 50  0001 C CNN
+F 1 "Logo_Open_Hardware_Small" H 6900 1425 50  0001 C CNN
+F 2 "durango:jaqueria" H 6900 1650 50  0001 C CNN
+F 3 "~" H 6900 1650 50  0001 C CNN
+	1    6900 1650
+	1    0    0    -1
+$EndComp
+$Comp
+L Jumper:Jumper_3_Bridged12 JP1
+U 1 1 6484669E
+P 7000 3500
+F 0 "JP1" V 7046 3567 50  0000 L CNN
+F 1 "16/32K" V 6955 3567 50  0000 L CNN
+F 2 "Jumper:SolderJumper-3_P1.3mm_Bridged12_RoundedPad1.0x1.5mm" H 7000 3500 50  0001 C CNN
+F 3 "~" H 7000 3500 50  0001 C CNN
+	1    7000 3500
+	0    -1   -1   0
+$EndComp
+$Comp
+L Memory_EPROM:27C080 U1
+U 1 1 64874267
+P 5500 2650
+F 0 "U1" H 5250 3900 50  0000 C CNN
+F 1 "27C010-080" H 5800 3900 50  0000 C CNN
+F 2 "Package_DIP:DIP-32_W15.24mm" H 5500 2650 50  0001 C CNN
+F 3 "http://ww1.microchip.com/downloads/en/devicedoc/doc0360.pdf" H 5500 2650 50  0001 C CNN
+	1    5500 2650
+	1    0    0    -1
+$EndComp
+Connection ~ 2350 3400
+Wire Wire Line
+	5500 3950 5500 4700
+Wire Wire Line
+	2850 5000 5100 5000
+Wire Wire Line
+	5100 5000 5100 3750
+Wire Wire Line
+	2800 5100 4800 5100
+Wire Wire Line
+	4800 5100 4800 3650
+Wire Wire Line
+	4800 3650 5100 3650
+Wire Wire Line
+	4400 1850 4600 1850
+Wire Wire Line
+	4600 1850 4600 3250
+Wire Wire Line
+	4600 3250 5100 3250
+Text Label 4400 1850 0    50   ~ 0
+BA3
+Text Label 5050 3250 2    50   ~ 0
+BA3
+Entry Wire Line
+	3050 1750 3150 1850
+Entry Wire Line
+	3050 1850 3150 1950
+Entry Wire Line
+	3050 1950 3150 2050
+Wire Wire Line
+	3150 1850 3400 1850
+Wire Wire Line
+	3150 1950 3400 1950
+Wire Wire Line
+	3150 2050 3400 2050
+Text Label 3200 1950 0    50   ~ 0
+D4
+Text Label 3200 2050 0    50   ~ 0
+D5
+Text Label 3200 1850 0    50   ~ 0
+D3
+Wire Wire Line
+	1700 2950 1950 2950
+Text Label 1750 2950 0    50   ~ 0
+A14
+Entry Wire Line
+	1600 2850 1700 2950
 Wire Bus Line
 	6250 1000 6250 2150
@@
 Wire Bus Line
 	1600 950  1600 4100
-$Comp
-L Graphic:Logo_Open_Hardware_Small LOGO1
-U 1 1 6483E578
-P 6900 1650
-F 0 "LOGO1" H 6900 1925 50  0001 C CNN
-F 1 "Logo_Open_Hardware_Small" H 6900 1425 50  0001 C CNN
-F 2 "durango:jaqueria" H 6900 1650 50  0001 C CNN
-F 3 "~" H 6900 1650 50  0001 C CNN
-	1    6900 1650
-	1    0    0    -1
-$EndComp
+Text Label 5100 3350 2    50   ~ 0
+MA18
+Text Label 5100 3450 2    50   ~ 0
+MA19
+Connection ~ 3900 3400
+Text Label 4400 1950 0    50   ~ 0
+BA4
+Text Label 4400 2050 0    50   ~ 0
+BA5
+$Comp
+L Jumper:Jumper_3_Bridged12 JP2
+U 1 1 648D7A9C
+P 7000 4500
+F 0 "JP2" V 7046 4567 50  0000 L CNN
+F 1 "040+" V 6955 4567 50  0000 L CNN
+F 2 "Jumper:SolderJumper-3_P1.3mm_Bridged12_RoundedPad1.0x1.5mm" H 7000 4500 50  0001 C CNN
+F 3 "~" H 7000 4500 50  0001 C CNN
+	1    7000 4500
+	0    -1   -1   0
+$EndComp
+$Comp
+L Jumper:Jumper_3_Bridged12 JP3
+U 1 1 648DA578
+P 7000 5500
+F 0 "JP3" V 7046 5567 50  0000 L CNN
+F 1 "080" V 6955 5567 50  0000 L CNN
+F 2 "Jumper:SolderJumper-3_P1.3mm_Bridged12_RoundedPad1.0x1.5mm" H 7000 5500 50  0001 C CNN
+F 3 "~" H 7000 5500 50  0001 C CNN
+	1    7000 5500
+	0    -1   -1   0
+$EndComp
+Text Label 7150 3500 0    50   ~ 0
+MA14
+Text Label 7150 4500 0    50   ~ 0
+MA18
+Text Label 7150 5500 0    50   ~ 0
+MA19
+$Comp
+L power:+5V #PWR0106
+U 1 1 648DB8D4
+P 7000 4750
+F 0 "#PWR0106" H 7000 4600 50  0001 C CNN
+F 1 "+5V" V 7015 4878 50  0000 L CNN
+F 2 "" H 7000 4750 50  0001 C CNN
+F 3 "" H 7000 4750 50  0001 C CNN
+	1    7000 4750
+	0    -1   -1   0
+$EndComp
+$Comp
+L power:+5V #PWR0107
+U 1 1 648DBECA
+P 7000 5750
+F 0 "#PWR0107" H 7000 5600 50  0001 C CNN
+F 1 "+5V" V 7015 5878 50  0000 L CNN
+F 2 "" H 7000 5750 50  0001 C CNN
+F 3 "" H 7000 5750 50  0001 C CNN
+	1    7000 5750
+	0    -1   -1   0
+$EndComp
+Text Label 7000 3750 3    50   ~ 0
+A14
+Text Label 7000 3250 2    50   ~ 0
+BA0
+Text Label 7000 4250 2    50   ~ 0
+BA4
+Text Label 7000 5250 2    50   ~ 0
+BA5
 $EndSCHEMATC
