File: hard/kicad/nanoLink/nanoLink.sch (KiCad schematic (older format))
At the start: 8 parts, among them J1 IOx, J2 nanoLink, U1 74HC139, U2 74HC174

Commit message: rework nanoLink interface PCB
Parts:
- removed U1: 74HC139, Package_DIP:DIP-16_W7.62mm_Socket, symbol 74xx:74LS139
- added U1: 74HC138, Package_DIP:DIP-16_W7.62mm_Socket, symbol 74xx:74LS138
- C1: value C -> 68pF; footprint Capacitor_THT:C_Rect_L7.0mm_W2.0mm_P5.00mm -> Capacitor_THT:C_Disc_D3.8mm_W2.6mm_P2.50mm
- R1: value R -> 6K8
Connections:
- net labels added: BA0
- net labels removed: ~SEL
- wire segments 39 -> 36
Other:
- moved on the sheet: J1, J2

Commit message: revised logos on nanoLink board
Parts:
- LOGO2: footprint durango:jaqueria -> durango:j300
Changed lines of the file:
@@
 F 0 "LOGO2" H 6200 2175 50  0001 C CNN
 F 1 "Logo_Open_Hardware_Small" H 6200 1675 50  0001 C CNN
-F 2 "durango:jaqueria" H 6200 1900 50  0001 C CNN
+F 2 "durango:j300" H 6200 1900 50  0001 C CNN
 F 3 "~" H 6200 1900 50  0001 C CNN
 	1    6200 1900
