File: hard/kicad/rosario/rosario.sch (KiCad schematic (older format))
At the start: 38 parts, among them J1 CARTRIDGE, J2 VIAport, J3 IOx, J4 nanoLink, J5 VDU, J6 POWER, J7 (6502), Q1 BC548, Q2 BC548, SW1 RESET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

Commit message: first complete routing for Rosario
Parts:
- added Q3: BC548, Package_TO_SOT_THT:TO-92_Inline, symbol Transistor_BJT:BC548
- D1: footprint Diode_THT:D_DO-35_SOD27_P2.54mm_Vertical_KathodeUp -> Diode_THT:D_DO-35_SOD27_P2.54mm_Vertical_AnodeUp
Connections:
- net +5V: now also Q3.1 (C); no longer J2.12 (Pin_12), J2.38 (Pin_38)
- net A0: now also U1.19 (Q0)
- net A1: now also U1.18 (Q1)
- net A2: now also U1.17 (Q2)
- net A3: now also U1.16 (Q3)
- net A4: now also U1.15 (Q4)
- net A5: now also U1.14 (Q5)
- net A6: now also U1.13 (Q6)
- net A7: now also U1.12 (Q7)
- net GND: now also BZ1.2 (+)
- net PB7: now also Q3.2 (B)
- net SC_RX: no longer RN3.4 (R3)
- net SC_TX: no longer RN3.5 (R4)
- net BZ: now reaches BZ1.1 (-)
- net BZ: now also Q3.3 (E)
- new net CA2: J2.12 (Pin_12), RN3.4 (R3)
- new net CB2: J2.38 (Pin_38), RN3.5 (R4)
- no-connect marks 12 -> 15
Other:
- moved on the sheet: BZ1, J5

Commit message: definitive Rosario v1
Parts:
- added JP1: ROM, Jumper:SolderJumper-3_P1.3mm_Bridged12_RoundedPad1.0x1.5mm, symbol Jumper:Jumper_3_Bridged12
- added JP2: 32K, Jumper:SolderJumper-3_P1.3mm_Bridged12_RoundedPad1.0x1.5mm, symbol Jumper:Jumper_3_Bridged12
- added R4: 33, Resistor_THT:R_Axial_DIN0309_L9.0mm_D3.2mm_P2.54mm_Vertical, symbol Device:R
- U3: value 62256 -> 62256 / 27C256
Connections:
- net A14: now also JP2.3 (B)
- net A15: now also JP1.1 (A); no longer U3.20 (~CS)
- net BZ: now also R4.1; no longer BZ1.1 (-)
- net ROM_~CS: now also JP1.3 (B)
- net ~WE: now also JP2.1 (A); no longer U3.27 (~WE~)
- new net BZR: BZ1.1 (-), R4.2
- new net RAM_~CS: JP1.2 (C), U3.20 (~CS)
- new net RAM_~WE: JP2.2 (C), U3.27 (~WE~)
Other:
- moved on the sheet: BZ1
Changed lines of the file:
@@
 P 6600 3050
 F 0 "U3" H 6600 3050 50  0000 C CNN
-F 1 "62256" H 6800 4150 50  0000 C CNN
+F 1 "62256 / 27C256" H 6950 4150 50  0000 C CNN
 F 2 "Package_DIP:DIP-28_W15.24mm_Socket" H 6600 3050 50  0001 C CNN
 F 3 "http://www.6502.org/users/alexis/62256.pdf" H 6600 3050 50  0001 C CNN
@@
 L Device:Buzzer BZ1
 U 1 1 652DC822
-P 1250 7050
-F 0 "BZ1" H 1402 7079 50  0000 L CNN
-F 1 "Buzzer" H 1402 6988 50  0000 L CNN
-F 2 "Buzzer_Beeper:Buzzer_12x9.5RM7.6" V 1225 7150 50  0001 C CNN
-F 3 "~" V 1225 7150 50  0001 C CNN
-	1    1250 7050
+P 1650 7050
+F 0 "BZ1" H 1802 7079 50  0000 L CNN
+F 1 "Buzzer" H 1802 6988 50  0000 L CNN
+F 2 "Buzzer_Beeper:Buzzer_12x9.5RM7.6" V 1625 7150 50  0001 C CNN
+F 3 "~" V 1625 7150 50  0001 C CNN
+	1    1650 7050
 	1    0    0    -1
 $EndComp
@@
 Wire Wire Line
 	6000 2150 5800 2150
-Text Label 7750 4600 0    50   ~ 0
+Text Label 5400 5500 0    50   ~ 0
 ~WE
 $Comp
@@
 Text Label 8300 5900 2    50   ~ 0
 R~W
-Text Label 8300 5000 2    50   ~ 0
+Text Label 8150 4900 0    50   ~ 0
 A15
 Text Label 8900 5800 0    50   ~ 0
@@
 Wire Wire Line
 	8350 2950 8050 2950
-Wire Wire Line
-	8050 2950 8050 4600
-Text Label 8050 5500 0    50   ~ 0
+Text Label 8100 5500 0    50   ~ 0
 ~WE
 Wire Wire Line
@@
 Text Label 2000 1750 0    50   ~ 0
 ~IRQ
-Wire Wire Line
-	8050 4600 6000 4600
-Connection ~ 8050 4600
-Wire Wire Line
-	8050 4600 8050 5500
-Wire Wire Line
-	6000 4600 6000 3950
 Text Label 8200 4650 0    50   ~ 0
 ~OE
@@
 	10550 3450 10800 3450
 Wire Wire Line
-	8150 5000 5750 5000
-Wire Wire Line
-	5750 5000 5750 3750
+	5750 4850 5750 3750
 Wire Wire Line
 	5750 3750 6000 3750
-Connection ~ 8150 5000
 Text Label 10800 2650 2    50   ~ 0
 D0
@@
 L power:GND #PWR0135
 U 1 1 661C5E1B
-P 1150 7150
-F 0 "#PWR0135" H 1150 6900 50  0001 C CNN
-F 1 "GND" H 1155 6977 50  0000 C CNN
-F 2 "" H 1150 7150 50  0001 C CNN
-F 3 "" H 1150 7150 50  0001 C CNN
-	1    1150 7150
+P 1550 7150
+F 0 "#PWR0135" H 1550 6900 50  0001 C CNN
+F 1 "GND" H 1555 6977 50  0000 C CNN
+F 2 "" H 1550 7150 50  0001 C CNN
+F 3 "" H 1550 7150 50  0001 C CNN
+	1    1550 7150
 	1    0    0    -1
 $EndComp
@@
 P 5250 2850
 F 0 "J5" H 5250 3850 50  0000 C CNN
-F 1 "VDU" H 5250 1750 50  0000 C CNN
+F 1 "VDU" H 5400 1850 50  0000 C CNN
 F 2 "Connector_PinSocket_2.54mm:PinSocket_1x20_P2.54mm_Vertical" H 5250 2850 50  0001 C CNN
 F 3 "~" H 5250 2850 50  0001 C CNN
@@
 Wire Wire Line
 	5450 3850 5600 3850
-Wire Bus Line
-	1850 3600 1850 4250
-Wire Bus Line
-	9100 3950 9100 4450
-Wire Bus Line
-	10350 1600 10350 3650
-Wire Bus Line
-	800  1800 800  2500
-Wire Bus Line
-	10600 1700 10600 3250
-Wire Bus Line
-	2150 4250 2150 5350
-Wire Bus Line
-	2100 1600 2100 2750
-Wire Bus Line
-	650  4250 650  5350
-Wire Bus Line
-	3800 1700 3800 2750
-Wire Bus Line
-	3550 1700 3550 2750
-Wire Bus Line
-	1950 900  1950 1800
-Wire Bus Line
-	650  900  650  4250
-Wire Bus Line
-	5700 1600 5700 3750
-Wire Bus Line
-	7400 1700 7400 4450
-Wire Bus Line
-	7500 1600 7500 3750
-Wire Bus Line
-	1950 1800 1950 4250
 Text Label 5000 2150 0    50   ~ 0
 A0
@@
 Text Label 5000 2850 0    50   ~ 0
 A7
+$Comp
+L Jumper:Jumper_3_Bridged12 JP1
+U 1 1 6614823B
+P 5750 5000
+F 0 "JP1" H 5750 5111 50  0000 C CNN
+F 1 "ROM" H 6000 5150 50  0000 C CNN
+F 2 "Jumper:SolderJumper-3_P1.3mm_Bridged12_RoundedPad1.0x1.5mm" H 5750 5000 50  0001 C CNN
+F 3 "~" H 5750 5000 50  0001 C CNN
+	1    5750 5000
+	-1   0    0    1
+$EndComp
+Wire Wire Line
+	8150 5000 6000 5000
+Connection ~ 8150 5000
+Text Label 5500 5000 2    50   ~ 0
+ROM_~CS
+Text Label 5750 4800 2    50   ~ 0
+RAM_~CS
+Wire Wire Line
+	8050 2950 8050 5500
+Text Label 6000 5000 0    50   ~ 0
+A15
+$Comp
+L Jumper:Jumper_3_Bridged12 JP2
+U 1 1 66191023
+P 5150 5500
+F 0 "JP2" H 5150 5611 50  0000 C CNN
+F 1 "32K" H 5400 5650 50  0000 C CNN
+F 2 "Jumper:SolderJumper-3_P1.3mm_Bridged12_RoundedPad1.0x1.5mm" H 5150 5500 50  0001 C CNN
+F 3 "~" H 5150 5500 50  0001 C CNN
+	1    5150 5500
+	-1   0    0    1
+$EndComp
+Wire Wire Line
+	6000 3950 5150 3950
+Wire Wire Line
+	5150 3950 5150 5350
+Wire Wire Line
+	8050 5500 5400 5500
+Connection ~ 8050 5500
+Text Label 4900 5500 2    50   ~ 0
+A14
+Text Label 5150 5350 2    50   ~ 0
+RAM_~WE
+$Comp
+L Device:R R4
+U 1 1 662654C3
+P 1300 6950
+F 0 "R4" V 1400 6900 50  0000 L CNN
+F 1 "33" V 1300 6950 50  0000 C CNN
+F 2 "Resistor_THT:R_Axial_DIN0309_L9.0mm_D3.2mm_P2.54mm_Vertical" V 1230 6950 50  0001 C CNN
+F 3 "~" H 1300 6950 50  0001 C CNN
+	1    1300 6950
+	0    -1   1    0
+$EndComp
+Wire Wire Line
+	1450 6950 1550 6950
+Text Label 1550 6950 3    50   ~ 0
+BZR
+Wire Bus Line
+	1850 3600 1850 4250
+Wire Bus Line
+	9100 3950 9100 4450
+Wire Bus Line
+	10350 1600 10350 3650
+Wire Bus Line
+	800  1800 800  2500
+Wire Bus Line
+	10600 1700 10600 3250
+Wire Bus Line
+	2150 4250 2150 5350
+Wire Bus Line
+	2100 1600 2100 2750
+Wire Bus Line
+	650  4250 650  5350
+Wire Bus Line
+	3800 1700 3800 2750
+Wire Bus Line
+	3550 1700 3550 2750
+Wire Bus Line
+	1950 900  1950 1800
+Wire Bus Line
+	650  900  650  4250
+Wire Bus Line
+	5700 1600 5700 3750
+Wire Bus Line
+	7400 1700 7400 4450
+Wire Bus Line
+	7500 1600 7500 3750
+Wire Bus Line
+	1950 1800 1950 4250
 $EndSCHEMATC

Commit message: upgrade Rosario to v1.1
Parts:
- added Q4: BC558, Package_TO_SOT_THT:TO-92_Inline, symbol Transistor_BJT:BC558
- added R6: 3K3, Resistor_THT:R_Axial_DIN0207_L6.3mm_D2.5mm_P2.54mm_Vertical, symbol Device:R
- J2: value VIAport -> VIAport (PB = output only)
- RN3: value 22K -> 4K7
Connections:
- net +5V: now also RN3.1 (common); no longer R3.2
- net GND: now also R3.2, Q4.1 (C), R6.2; no longer BZ1.2 (+), RN3.1 (common)
- net IOSEL: now also R6.1; no longer RN3.2 (R1)
- net P21: now also RN3.2 (R1); no longer R3.1
- net PB7: now also Q4.2 (B); no longer Q3.2 (B)
- net SC_CL: now also R3.1; no longer RN3.3 (R2)
- net SC_RX: now also RN3.5 (R4)
- net SC_TX: now also J2.38 (Pin_38), Q3.2 (B), RN3.3 (R2)
- removed net CB2: J2.38 (Pin_38), RN3.5 (R4)
- new net BZG: BZ1.2 (+), Q4.3 (E)
Other:
- moved on the sheet: BZ1, Q3, R3, R4, RN3
Changed lines of the file:
@@
 P 1250 3000
 F 0 "J2" H 1300 4117 50  0000 C CNN
-F 1 "VIAport" H 1300 4026 50  0000 C CNN
+F 1 "VIAport (PB = output only)" H 1300 4026 50  0000 C CNN
 F 2 "Connector_IDC:IDC-Header_2x20_P2.54mm_Vertical" H 1250 3000 50  0001 C CNN
 F 3 "~" H 1250 3000 50  0001 C CNN
@@
 L Device:Buzzer BZ1
 U 1 1 652DC822
-P 1650 7050
-F 0 "BZ1" H 1802 7079 50  0000 L CNN
-F 1 "Buzzer" H 1802 6988 50  0000 L CNN
-F 2 "Buzzer_Beeper:Buzzer_12x9.5RM7.6" V 1625 7150 50  0001 C CNN
-F 3 "~" V 1625 7150 50  0001 C CNN
-	1    1650 7050
+P 1950 7050
+F 0 "BZ1" H 2102 7079 50  0000 L CNN
+F 1 "Buzzer" H 2102 6988 50  0000 L CNN
+F 2 "Buzzer_Beeper:Buzzer_12x9.5RM7.6" V 1925 7150 50  0001 C CNN
+F 3 "~" V 1925 7150 50  0001 C CNN
+	1    1950 7050
 	1    0    0    -1
 $EndComp
@@
 L Device:R_Network04 RN3
 U 1 1 667CBFEE
-P 4100 1300
-F 0 "RN3" V 3800 1200 50  0000 L CNN
-F 1 "22K" V 4300 1200 50  0000 L CNN
-F 2 "Resistor_THT:R_Array_SIP5" V 4375 1300 50  0001 C CNN
-F 3 "http://www.vishay.com/docs/31509/csc.pdf" H 4100 1300 50  0001 C CNN
-	1    4100 1300
+P 4400 950
+F 0 "RN3" V 4100 850 50  0000 L CNN
+F 1 "4K7" V 4600 850 50  0000 L CNN
+F 2 "Resistor_THT:R_Array_SIP5" V 4675 950 50  0001 C CNN
+F 3 "http://www.vishay.com/docs/31509/csc.pdf" H 4400 950 50  0001 C CNN
+	1    4400 950
 	0    1    1    0
 $EndComp
@@
 Text Label 3350 3250 0    50   ~ 0
 SC_CL
-Text Label 3900 1200 2    50   ~ 0
+Text Label 3600 850  2    50   ~ 0
 SC_CL
-Text Label 3900 1300 2    50   Italic 0
-CA2
-Text Label 3900 1400 2    50   Italic 0
-CB2
-Wire Wire Line
-	3900 1100 3600 1100
-Connection ~ 3600 1100
 Wire Wire Line
 	3350 3250 3650 3250
 Wire Wire Line
-	3650 3250 3650 1200
-Wire Wire Line
-	3650 1200 3900 1200
+	3650 3250 3650 1500
 Text Label 3350 3550 0    50   ~ 0
 XT
 Text Label 3400 3750 3    50   ~ 0
 EXT
-$Comp
-L power:GND #PWR0114
-U 1 1 66806929
-P 4300 1100
-F 0 "#PWR0114" H 4300 850 50  0001 C CNN
-F 1 "GND" V 4200 1000 50  0000 C CNN
-F 2 "" H 4300 1100 50  0001 C CNN
-F 3 "" H 4300 1100 50  0001 C CNN
-	1    4300 1100
-	0    -1   -1   0
-$EndComp
 Wire Wire Line
 	3500 5850 2600 5850
@@
 L Device:R R3
 U 1 1 66D4CE79
-P 3050 1200
-F 0 "R3" V 3150 1150 50  0000 L CNN
-F 1 "3K3" V 3050 1200 50  0000 C CNN
-F 2 "Resistor_THT:R_Axial_DIN0207_L6.3mm_D2.5mm_P2.54mm_Vertical" V 2980 1200 50  0001 C CNN
-F 3 "~" H 3050 1200 50  0001 C CNN
-	1    3050 1200
-	0    1    1    0
+P 3750 850
+F 0 "R3" V 3850 800 50  0000 L CNN
+F 1 "3K3" V 3750 850 50  0000 C CNN
+F 2 "Resistor_THT:R_Axial_DIN0207_L6.3mm_D2.5mm_P2.54mm_Vertical" V 3680 850 50  0001 C CNN
+F 3 "~" H 3750 850 50  0001 C CNN
+	1    3750 850
+	0    -1   -1   0
 $EndComp
 $Comp
@@
 Wire Wire Line
 	2900 1100 2900 1200
-Text Label 3200 1200 0    50   ~ 0
+Text Label 4200 750  2    50   ~ 0
 P21
 $Comp
@@
 	10550 2350 10800 2350
 Connection ~ 10550 2150
-Connection ~ 2900 1200
 $Comp
 L Transistor_BJT:BC548 Q3
 U 1 1 661C246B
-P 1000 6750
-F 0 "Q3" H 1191 6796 50  0000 L CNN
-F 1 "BC548" H 1191 6705 50  0000 L CNN
-F 2 "Package_TO_SOT_THT:TO-92_Inline" H 1200 6675 50  0001 L CIN
-F 3 "http://www.fairchildsemi.com/ds/BC/BC547.pdf" H 1000 6750 50  0001 L CNN
-	1    1000 6750
+P 1300 6750
+F 0 "Q3" H 1491 6796 50  0000 L CNN
+F 1 "BC548" H 1491 6705 50  0000 L CNN
+F 2 "Package_TO_SOT_THT:TO-92_Inline" H 1500 6675 50  0001 L CIN
+F 3 "http://www.fairchildsemi.com/ds/BC/BC547.pdf" H 1300 6750 50  0001 L CNN
+	1    1300 6750
 	1    0    0    -1
 $EndComp
@@
 L power:GND #PWR0135
 U 1 1 661C5E1B
-P 1550 7150
-F 0 "#PWR0135" H 1550 6900 50  0001 C CNN
-F 1 "GND" H 1555 6977 50  0000 C CNN
-F 2 "" H 1550 7150 50  0001 C CNN
-F 3 "" H 1550 7150 50  0001 C CNN
-	1    1550 7150
-	1    0    0    -1
-$EndComp
-Wire Wire Line
-	1150 6950 1100 6950
-Text Label 1100 6950 3    50   ~ 0
+P 600 7150
+F 0 "#PWR0135" H 600 6900 50  0001 C CNN
+F 1 "GND" V 700 7100 50  0000 C CNN
+F 2 "" H 600 7150 50  0001 C CNN
+F 3 "" H 600 7150 50  0001 C CNN
+	1    600  7150
+	0    1    1    0
+$EndComp
+Wire Wire Line
+	1450 6950 1400 6950
+Text Label 1400 6950 3    50   ~ 0
 BZ
 Wire Wire Line
-	800  5450 800  6750
+	800  5450 800  6850
 Connection ~ 800  5450
 Wire Wire Line
@@
 L power:+5V #PWR0136
 U 1 1 6620B728
-P 1100 6550
-F 0 "#PWR0136" H 1100 6400 50  0001 C CNN
-F 1 "+5V" H 1115 6723 50  0000 C CNN
-F 2 "" H 1100 6550 50  0001 C CNN
-F 3 "" H 1100 6550 50  0001 C CNN
-	1    1100 6550
+P 1400 6550
+F 0 "#PWR0136" H 1400 6400 50  0001 C CNN
+F 1 "+5V" H 1415 6723 50  0000 C CNN
+F 2 "" H 1400 6550 50  0001 C CNN
+F 3 "" H 1400 6550 50  0001 C CNN
+	1    1400 6550
 	1    0    0    -1
 $EndComp
@@
 Text Label 1550 2600 0    50   Italic 0
 CA2
-Text Label 1550 3900 0    50   Italic 0
-CB2
 Connection ~ 5550 1650
 Connection ~ 5500 1750
@@
 L Device:R R4
 U 1 1 662654C3
-P 1300 6950
-F 0 "R4" V 1400 6900 50  0000 L CNN
-F 1 "33" V 1300 6950 50  0000 C CNN
-F 2 "Resistor_THT:R_Axial_DIN0309_L9.0mm_D3.2mm_P2.54mm_Vertical" V 1230 6950 50  0001 C CNN
-F 3 "~" H 1300 6950 50  0001 C CNN
-	1    1300 6950
+P 1600 6950
+F 0 "R4" V 1700 6900 50  0000 L CNN
+F 1 "33" V 1600 6950 50  0000 C CIN
+F 2 "Resistor_THT:R_Axial_DIN0309_L9.0mm_D3.2mm_P2.54mm_Vertical" V 1530 6950 50  0001 C CNN
+F 3 "~" H 1600 6950 50  0001 C CNN
+	1    1600 6950
 	0    -1   1    0
 $EndComp
 Wire Wire Line
-	1450 6950 1550 6950
-Text Label 1550 6950 3    50   ~ 0
+	1750 6950 1850 6950
+Text Label 1850 6950 3    50   ~ 0
 BZR
+$Comp
+L Transistor_BJT:BC558 Q4
+U 1 1 66178C1F
+P 800 7050
+F 0 "Q4" V 1035 7050 50  0000 C CNN
+F 1 "BC558" V 1126 7050 50  0000 C CNN
+F 2 "Package_TO_SOT_THT:TO-92_Inline" H 1000 6975 50  0001 L CIN
+F 3 "http://www.fairchildsemi.com/ds/BC/BC557.pdf" H 800 7050 50  0001 L CNN
+	1    800  7050
+	0    -1   1    0
+$EndComp
+Wire Wire Line
+	1000 7150 1850 7150
+Text Label 1100 6750 1    50   ~ 0
+SC_TX
+Text Label 1850 7150 3    50   ~ 0
+BZG
+Text Label 1550 3900 0    50   ~ 0
+SC_TX
+$Comp
+L Device:R R6
+U 1 1 662226AF
+P 3750 1100
+F 0 "R6" V 3650 1050 50  0000 L CNN
+F 1 "3K3" V 3750 1100 50  0000 C CNN
+F 2 "Resistor_THT:R_Axial_DIN0207_L6.3mm_D2.5mm_P2.54mm_Vertical" V 3680 1100 50  0001 C CNN
+F 3 "~" H 3750 1100 50  0001 C CNN
+	1    3750 1100
+	0    -1   1    0
+$EndComp
+Connection ~ 3600 1100
+$Comp
+L power:GND #PWR0114
+U 1 1 662291D7
+P 3900 1100
+F 0 "#PWR0114" H 3900 850 50  0001 C CNN
+F 1 "GND" H 3905 927 50  0000 C CNN
+F 2 "" H 3900 1100 50  0001 C CNN
+F 3 "" H 3900 1100 50  0001 C CNN
+	1    3900 1100
+	1    0    0    -1
+$EndComp
+Wire Wire Line
+	3900 850  3900 1100
+Connection ~ 3900 1100
+$Comp
+L power:+5V #PWR0137
+U 1 1 6628EBFF
+P 4600 750
+F 0 "#PWR0137" H 4600 600 50  0001 C CNN
+F 1 "+5V" H 4615 923 50  0000 C CNN
+F 2 "" H 4600 750 50  0001 C CNN
+F 3 "" H 4600 750 50  0001 C CNN
+	1    4600 750
+	1    0    0    -1
+$EndComp
+Text Label 4200 850  2    50   ~ 0
+SC_TX
+Text Label 4200 1050 2    50   ~ 0
+SC_RX
+Text Label 4200 950  2    50   Italic 0
+CA2
 Wire Bus Line
 	1850 3600 1850 4250

Commit message: use both 573 on Rosario
Parts:
- U5: value 74HC574 -> 74HC573/4; symbol 74xx:74LS574 -> 74xx:74LS573
Changed lines of the file:
@@
 Wire Bus Line
 	3550 1700 3800 1700
-$Comp
-L 74xx:74LS574 U5
-U 1 1 6691BB95
-P 1400 5250
-F 0 "U5" H 1400 5300 50  0000 C CNN
-F 1 "74HC574" H 1200 5900 50  0000 C CNN
-F 2 "Package_DIP:DIP-20_W7.62mm_Socket" H 1400 5250 50  0001 C CNN
-F 3 "http://www.ti.com/lit/gpn/sn74LS574" H 1400 5250 50  0001 C CNN
-	1    1400 5250
-	-1   0    0    -1
-$EndComp
 Text Label 1900 4750 0    50   ~ 0
 PA0
@@
 	1    0    0    -1
 $EndComp
-Connection ~ 1400 6050
 Wire Wire Line
 	1550 4000 1550 4450
@@
 Text Label 4200 950  2    50   Italic 0
 CA2
+Connection ~ 1400 6050
+Wire Bus Line
+	10600 1700 10600 3250
+Wire Bus Line
+	2150 4250 2150 5350
+Wire Bus Line
+	2100 1600 2100 2750
+Wire Bus Line
+	650  4250 650  5350
+Wire Bus Line
+	9100 3950 9100 4450
+Wire Bus Line
+	7500 1600 7500 3750
+Wire Bus Line
+	7400 1700 7400 4450
+Wire Bus Line
+	10350 1600 10350 3650
+Wire Bus Line
+	5700 1600 5700 3750
+Wire Bus Line
+	3800 1700 3800 2750
+Wire Bus Line
+	3550 1700 3550 2750
+Wire Bus Line
+	800  1800 800  2500
 Wire Bus Line
 	1850 3600 1850 4250
 Wire Bus Line
-	9100 3950 9100 4450
-Wire Bus Line
-	10350 1600 10350 3650
-Wire Bus Line
-	800  1800 800  2500
-Wire Bus Line
-	10600 1700 10600 3250
-Wire Bus Line
-	2150 4250 2150 5350
-Wire Bus Line
-	2100 1600 2100 2750
-Wire Bus Line
-	650  4250 650  5350
-Wire Bus Line
-	3800 1700 3800 2750
-Wire Bus Line
-	3550 1700 3550 2750
-Wire Bus Line
 	1950 900  1950 1800
 Wire Bus Line
+	1950 1800 1950 4250
+Wire Bus Line
 	650  900  650  4250
-Wire Bus Line
-	5700 1600 5700 3750
-Wire Bus Line
-	7400 1700 7400 4450
-Wire Bus Line
-	7500 1600 7500 3750
-Wire Bus Line
-	1950 1800 1950 4250
+$Comp
+L 74xx:74LS573 U5
+U 1 1 6691BB95
+P 1400 5250
+F 0 "U5" H 1400 5300 50  0000 C CNN
+F 1 "74HC573/4" H 1150 5900 50  0000 C CNN
+F 2 "Package_DIP:DIP-20_W7.62mm_Socket" H 1400 5250 50  0001 C CNN
+F 3 "http://www.ti.com/lit/gpn/sn74LS574" H 1400 5250 50  0001 C CNN
+	1    1400 5250
+	-1   0    0    -1
+$EndComp
 $EndSCHEMATC

Commit message: cartridge silkscreen on Rosario
Parts:
- RN2: value 3K3 -> 22K
Changed lines of the file:
@@
 P 2350 1200
 F 0 "RN2" V 1733 1200 50  0000 C CNN
-F 1 "3K3" V 1824 1200 50  0000 C CNN
+F 1 "22K" V 1824 1200 50  0000 C CNN
 F 2 "Resistor_THT:R_Array_SIP9" V 2825 1200 50  0001 C CNN
 F 3 "http://www.vishay.com/docs/31509/csc.pdf" H 2350 1200 50  0001 C CNN
@@
 CA2
 Connection ~ 1400 6050
-Wire Bus Line
-	10600 1700 10600 3250
-Wire Bus Line
-	2150 4250 2150 5350
-Wire Bus Line
-	2100 1600 2100 2750
-Wire Bus Line
-	650  4250 650  5350
-Wire Bus Line
-	9100 3950 9100 4450
-Wire Bus Line
-	7500 1600 7500 3750
-Wire Bus Line
-	7400 1700 7400 4450
-Wire Bus Line
-	10350 1600 10350 3650
-Wire Bus Line
-	5700 1600 5700 3750
-Wire Bus Line
-	3800 1700 3800 2750
-Wire Bus Line
-	3550 1700 3550 2750
-Wire Bus Line
-	800  1800 800  2500
-Wire Bus Line
-	1850 3600 1850 4250
-Wire Bus Line
-	1950 900  1950 1800
-Wire Bus Line
-	1950 1800 1950 4250
-Wire Bus Line
-	650  900  650  4250
 $Comp
 L 74xx:74LS573 U5
@@
 	-1   0    0    -1
 $EndComp
+Wire Bus Line
+	1850 3600 1850 4250
+Wire Bus Line
+	9100 3950 9100 4450
+Wire Bus Line
+	10350 1600 10350 3650
+Wire Bus Line
+	800  1800 800  2500
+Wire Bus Line
+	10600 1700 10600 3250
+Wire Bus Line
+	2150 4250 2150 5350
+Wire Bus Line
+	2100 1600 2100 2750
+Wire Bus Line
+	650  4250 650  5350
+Wire Bus Line
+	3800 1700 3800 2750
+Wire Bus Line
+	3550 1700 3550 2750
+Wire Bus Line
+	1950 900  1950 1800
+Wire Bus Line
+	650  900  650  4250
+Wire Bus Line
+	5700 1600 5700 3750
+Wire Bus Line
+	7400 1700 7400 4450
+Wire Bus Line
+	7500 1600 7500 3750
+Wire Bus Line
+	1950 1800 1950 4250
 $EndSCHEMATC

Commit message: Rosario v1.2 and improve simpleIO
Connections:
- net SC_TX: now also RN3.4 (R3); no longer RN3.3 (R2)
- net ~IOX: now also J2.12 (Pin_12)
- removed net CA2: J2.12 (Pin_12), RN3.4 (R3)
- no-connect marks 15 -> 16
Changed lines of the file:
@@
 NoConn ~ 1050 3000
 NoConn ~ 1050 3100
-Text Label 1550 2600 0    50   Italic 0
-CA2
 Connection ~ 5550 1650
 Connection ~ 5500 1750
@@
 	1    0    0    -1
 $EndComp
-Text Label 4200 850  2    50   ~ 0
+Text Label 4200 950  2    50   ~ 0
 SC_TX
 Text Label 4200 1050 2    50   ~ 0
 SC_RX
-Text Label 4200 950  2    50   Italic 0
-CA2
 Connection ~ 1400 6050
 $Comp
@@
 	-1   0    0    -1
 $EndComp
+NoConn ~ 4200 850
 Wire Bus Line
 	1850 3600 1850 4250
@@
 Wire Bus Line
 	1950 1800 1950 4250
+Text Label 1550 2600 0    50   ~ 0
+~IOX
 $EndSCHEMATC
