File: hard/kicad/simple-io/simple-io.kicad_pcb (KiCad board)
At the start: 2 copper layers, 97.8 x 72.4 mm, 31 parts, among them J1 SS-22, J2 VIAport, J3 TTL SERIAL, SW1 PA0, SW2 PA1, SW3 PA2, SW4 PA3, SW5 PA4, SW6 PA5, SW7 PA6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

Commit message: Rosario v1.2 and improve simpleIO
Parts:
- moved D2 0.64 mm to (55.2, 68.6)
- moved D3 0.64 mm to (64.8, 68.6)
- moved D1 0.63 mm to (45.7, 68.6)
Routing:
- net /RB0: track 55.3 -> 56.6 mm
- net GND: track 511.0 -> 512.0 mm
- net /RB2: track 42.4 -> 43.0 mm
- net /RB1: track 43.2 -> 43.9 mm
Other:
- board text added: "(Chihuahua)"
- board text added: "(Rosario)"
Changed lines of the file:
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@@
   (general
     (thickness 1.6)
-    (drawings 36)
-    (tracks 515)
+    (drawings 38)
+    (tracks 520)
     (zones 0)
     (modules 31)
@@
   )
   (setup
-    (last_trace_width 0.635)
+    (last_trace_width 0.28)
     (user_trace_width 0.2)
     (user_trace_width 0.28)
@@
   )
   (module LED_THT:LED_D3.0mm (layer F.Cu)
-    (at 65.405 68.58 90)
+    (at 64.77 68.58 90)
     (descr "LED, diameter 3.0mm, 2 pins")
     (tags "LED diameter 3.0mm 2 pins")
@@
   )
   (module LED_THT:LED_D3.0mm (layer F.Cu)
-    (at 55.88 68.58 90)
+    (at 55.245 68.58 90)
     (descr "LED, diameter 3.0mm, 2 pins")
     (tags "LED diameter 3.0mm 2 pins")
@@
   )
   (module LED_THT:LED_D3.0mm (layer F.Cu)
-    (at 46.355 68.58 90)
+    (at 45.72 68.58 90)
     (descr "LED, diameter 3.0mm, 2 pins")
     (tags "LED diameter 3.0mm 2 pins")
@@
     )
   )
+  (gr_text "(Rosario)" (at 90.17 30.48) (layer F.SilkS)
+    (effects (font (size 1 1) (thickness 0.15)) (justify left))
+  )
+  (gr_text "(Chihuahua)" (at 45.085 31.115) (layer F.SilkS)
+    (effects (font (size 1 1) (thickness 0.15)) (justify right))
+  )
   (gr_text Rx (at 78.74 26.416) (layer B.SilkS)
     (effects (font (size 0.75 0.75) (thickness 0.15)) (justify mirror))
@@
   (segment (start 25.4 63.5) (end 24.13 62.23) (width 0.635) (layer F.Cu) (net 1))
   (segment (start 23.495 62.23) (end 22.225 62.23) (width 0.28) (layer F.Cu) (net 1))
-  (segment (start 46.355 68.58) (end 112.395 68.58) (width 0.635) (layer B.Cu) (net 1))
   (segment (start 22.86 90.17) (end 22.86 78.74) (width 0.635) (layer F.Cu) (net 1))
   (segment (start 28.575 95.885) (end 22.86 90.17) (width 0.635) (layer F.Cu) (net 1))
@@
   (segment (start 116.309684 66.200316) (end 113.93 68.58) (width 0.635) (layer F.Cu) (net 1))
   (segment (start 116.309684 41.805316) (end 116.309684 66.200316) (width 0.635) (layer F.Cu) (net 1))
-  (segment (start 46.355 70.115) (end 42.347499 74.122501) (width 0.635) (layer F.Cu) (net 1))
-  (segment (start 46.355 68.58) (end 46.355 70.115) (width 0.635) (layer F.Cu) (net 1))
   (segment (start 42.347499 95.447501) (end 41.91 95.885) (width 0.635) (layer F.Cu) (net 1))
   (segment (start 41.91 95.885) (end 46.355 95.885) (width 0.635) (layer F.Cu) (net 1))
@@
   (segment (start 112.395 84.455) (end 111.76 85.09) (width 0.635) (layer F.Cu) (net 1))
   (segment (start 112.395 68.58) (end 112.395 84.455) (width 0.635) (layer F.Cu) (net 1))
+  (segment (start 46.355 68.58) (end 46.99 68.58) (width 0.635) (layer B.Cu) (net 1))
+  (segment (start 46.99 68.58) (end 45.72 68.58) (width 0.635) (layer B.Cu) (net 1))
+  (segment (start 46.99 68.58) (end 112.395 68.58) (width 0.635) (layer B.Cu) (net 1))
+  (segment (start 45.72 70.75) (end 44.5825 71.8875) (width 0.635) (layer F.Cu) (net 1))
+  (segment (start 45.72 68.58) (end 45.72 70.75) (width 0.635) (layer F.Cu) (net 1))
+  (segment (start 44.5825 71.8875) (end 42.347499 74.122501) (width 0.635) (layer F.Cu) (net 1))
   (segment (start 19.685 66.675) (end 22.86 63.5) (width 0.635) (layer B.Cu) (net 2))
   (segment (start 19.685 78.74) (end 19.685 66.675) (width 0.635) (layer B.Cu) (net 2))
@@
   (via (at 85.09 58.76) (size 0.8) (drill 0.5) (layers F.Cu B.Cu) (net 24))
   (segment (start 52.460902 66.04) (end 47.627792 66.04) (width 0.635) (layer B.Cu) (net 24))
-  (segment (start 47.627792 66.04) (end 46.355 66.04) (width 0.635) (layer B.Cu) (net 24))
   (segment (start 59.740902 58.76) (end 52.460902 66.04) (width 0.635) (layer B.Cu) (net 24))
   (segment (start 85.09 58.76) (end 59.740902 58.76) (width 0.635) (layer B.Cu) (net 24))
@@
   (segment (start 86.36 45.72) (end 86.36 47.625) (width 0.635) (layer F.Cu) (net 24))
   (segment (start 85.09 48.895) (end 85.09 58.76) (width 0.635) (layer F.Cu) (net 24))
+  (segment (start 46.99 66.04) (end 45.72 66.04) (width 0.635) (layer B.Cu) (net 24))
+  (segment (start 47.627792 66.04) (end 46.99 66.04) (width 0.635) (layer B.Cu) (net 24))
+  (segment (start 46.99 66.04) (end 46.355 66.04) (width 0.635) (layer B.Cu) (net 24))
   (via (at 86.36 59.6275) (size 0.8) (drill 0.5) (layers F.Cu B.Cu) (net 25))
   (segment (start 86.36 49.53) (end 86.36 59.6275) (width 0.635) (layer F.Cu) (net 25))
-  (segment (start 62.2925 59.6275) (end 55.88 66.04) (width 0.635) (layer B.Cu) (net 25))
-  (segment (start 86.36 59.6275) (end 62.2925 59.6275) (width 0.635) (layer B.Cu) (net 25))
+  (segment (start 61.6575 59.6275) (end 55.245 66.04) (width 0.635) (layer B.Cu) (net 25))
+  (segment (start 62.9275 59.6275) (end 61.6575 59.6275) (width 0.635) (layer B.Cu) (net 25))
+  (segment (start 86.36 59.6275) (end 62.9275 59.6275) (width 0.635) (layer B.Cu) (net 25))
   (segment (start 90.17 51.435) (end 90.17 60.325) (width 0.635) (layer F.Cu) (net 26))
   (segment (start 90.167501 51.432501) (end 90.17 51.435) (width 0.635) (layer F.Cu) (net 26))
   (via (at 90.17 60.495) (size 0.8) (drill 0.5) (layers F.Cu B.Cu) (net 26))
   (segment (start 90.17 60.325) (end 90.17 60.495) (width 0.635) (layer F.Cu) (net 26))
-  (segment (start 70.95 60.495) (end 65.405 66.04) (width 0.635) (layer B.Cu) (net 26))
-  (segment (start 90.17 60.495) (end 70.95 60.495) (width 0.635) (layer B.Cu) (net 26))
   (segment (start 91.44 47.620002) (end 90.167501 48.892501) (width 0.635) (layer F.Cu) (net 26))
   (segment (start 91.44 45.72) (end 91.44 47.620002) (width 0.635) (layer F.Cu) (net 26))
   (segment (start 90.167501 48.892501) (end 90.167501 51.432501) (width 0.635) (layer F.Cu) (net 26))
+  (segment (start 70.315 60.495) (end 64.77 66.04) (width 0.635) (layer B.Cu) (net 26))
+  (segment (start 71.925 60.495) (end 70.315 60.495) (width 0.635) (layer B.Cu) (net 26))
+  (segment (start 90.17 60.495) (end 71.925 60.495) (width 0.635) (layer B.Cu) (net 26))
   (via (at 91.44 61.3625) (size 0.8) (drill 0.5) (layers F.Cu B.Cu) (net 27))
   (segment (start 91.44 50.8) (end 91.44 61.3625) (width 0.635) (layer F.Cu) (net 27))
@@
   (segment (start 70.485 74.295) (end 78.105 74.295) (width 0.28) (layer B.Cu) (net 37))
   (segment (start 62.865 83.185) (end 62.865 76.685) (width 0.28) (layer F.Cu) (net 38))
-  (segment (start 63.864999 50.435001) (end 63.970001 50.329999) (width 0.28) (layer F.Cu) (net 38))
-  (segment (start 63.970001 50.329999) (end 64.77 49.53) (width 0.28) (layer F.Cu) (net 38))
-  (segment (start 63.864999 75.685001) (end 63.864999 50.435001) (width 0.28) (layer F.Cu) (net 38))
-  (segment (start 62.865 76.685) (end 63.864999 75.685001) (width 0.28) (layer F.Cu) (net 38))
+  (segment (start 62.865 51.435) (end 64.77 49.53) (width 0.28) (layer F.Cu) (net 38))
+  (segment (start 62.865 76.685) (end 62.865 51.435) (width 0.28) (layer F.Cu) (net 38))
   (segment (start 43.815 83.185) (end 43.815 76.685) (width 0.28) (layer F.Cu) (net 39))
   (segment (start 43.815 76.685) (end 47.625 72.875) (width 0.28) (layer F.Cu) (net 39))
