File: hard/kicad/omronkbd/omronkbd.kicad_pcb (KiCad board)
At the start: 2 copper layers, 351.8 x 144.1 mm, 123 parts, among them J1 TO COMPUTER, J101 MD/VCS1, J102 MD/VCS2, J2 IOx, J201 NES 1, J202 NES 2, J3 IOx, SW1 1, SW10 0, SW11 Q, SW12 W, SW13 E, SW14 R, SW15 T, SW16 Y, SW17 U, SW18 I, SW19 O, SW2 2, SW20 P, SW21 A, SW22 S, SW23 D, SW24 F, SW25 G, SW26 H, SW27 J, SW28 K, SW29 L, SW3 3, SW30 ENTER, SW31 LSHIFT, SW32 Z, SW33 X, SW34 C, SW35 V, SW36 B, SW37 N, SW38 M, SW39 L-ALT, SW4 4, SW40 SPACE, SW41 ESC, SW42 PGUP, SW43 PGDN, SW44 LCTRL, SW45 ORD, SW46 TAB, SW47 CAPS, SW48 <, SW49 APOS, SW5 5, SW50 GRAVE, SW51 Ñ, SW52 COMMA, SW53 IEXCL, SW54 PLUS, SW55 ACUTE, SW56 DOT, SW57 DEL, SW58 BKSP, SW59 Ç, SW6 6, SW60 MINUS, SW61 UP, SW62 LEFT, SW63 DOWN, SW64 RIGHT, SW65 R-ALT, SW66 RSHIFT, SW67 RCTRL, SW7 7, SW8 8, SW9 9, U1 74HC138, U101 74HC245, U102 74HC245, U103 74HC174, U2 74HC574, U201 74HC595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

Commit message: finish stub for OMRON keyboard
Parts:
- added SW68: L-SP, Button_Switch_THT:SW_SPST_Omron_B3F-40xx, F.Cu at (72.0, 229.2)
- added SW69: R-SP, Button_Switch_THT:SW_SPST_Omron_B3F-40xx, F.Cu at (156.6, 229.2)
- SW1, SW10, SW11, SW12, SW13, SW14, SW15, SW16, SW17, SW18, SW19, SW2, SW20, SW21, SW22, SW23, SW24, SW25, SW26, SW27, SW28, SW29, SW3, SW32, SW33, SW34, SW35, SW36, SW37, SW38, SW4, SW41, SW42, SW43, SW45, SW48, SW49, SW5, SW50, SW51, SW52, SW53, SW54, SW55, SW56, SW57, SW59, SW6, SW60, SW61, SW62, SW63, SW64, SW7, SW8, SW9: footprint Button_Switch_Keyboard:SW_Cherry_MX_1.00u_PCB -> Button_Switch_THT:SW_SPST_Omron_B3F-40xx
- SW30: footprint Button_Switch_Keyboard:SW_Cherry_MX_ISOEnter_PCB -> Button_Switch_THT:SW_SPST_Omron_B3F-40xx
- SW31, SW47: footprint Button_Switch_Keyboard:SW_Cherry_MX_1.25u_PCB -> Button_Switch_THT:SW_SPST_Omron_B3F-40xx
- SW39, SW44, SW46, SW65, SW67: footprint Button_Switch_Keyboard:SW_Cherry_MX_1.50u_PCB -> Button_Switch_THT:SW_SPST_Omron_B3F-40xx
- SW40: footprint Button_Switch_Keyboard:SW_Cherry_MX_6.25u_PCB -> Button_Switch_THT:SW_SPST_Omron_B3F-40xx
- SW58: footprint Button_Switch_Keyboard:SW_Cherry_MX_2.00u_PCB -> Button_Switch_THT:SW_SPST_Omron_B3F-40xx
- SW66: footprint Button_Switch_Keyboard:SW_Cherry_MX_2.75u_PCB -> Button_Switch_THT:SW_SPST_Omron_B3F-40xx
- moved U201 157.5 mm to (163.2, 142.9)
- moved RN1 148.1 mm to (113.0, 131.4)
- moved RN101 131.6 mm to (186.7, 131.4)
- moved U101 131.6 mm to (186.7, 142.9)
- moved U202 131.1 mm to (217.2, 131.4)
- moved J101 122.9 mm to (201.1, 115.6)
- moved LOGO2 119.4 mm to (218.4, 156.2)
- moved RN2 105.0 mm to (240.0, 131.4)
- moved U102 105.0 mm to (240.0, 142.9)
- moved SW42 104.4 mm to (256.0, 163.2), turned to 90 degrees
- moved SW43 104.2 mm to (256.0, 179.5), turned to 90 degrees
- moved SW64 104.1 mm to (256.0, 229.2), turned to 90 degrees
- moved J102 101.6 mm to (254.8, 115.6)
- moved SW61 97.7 mm to (243.3, 212.7), turned to 90 degrees
- moved SW63 97.7 mm to (243.3, 229.2), turned to 90 degrees
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Other:
- board size 351.8 x 144.1 mm -> 250.8 x 130.2 mm
